File: Hardware/_autosave-LTC.sch (KiCad schematic (older format))
At the start: 64 parts, among them J10 Conn_01x01_Female, J11 Conn_01x01_Female, J12 Conn_01x01_Female, J6 Conn_01x01_Female, J7 Conn_01x01_Female, J8 Conn_01x01_Female, J9 Conn_01x01_Female, Q2 Q_PMOS_GSD, Q3 Q_PMOS_GSD, Q4 Q_PMOS_GSD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

Commit message: Save before ZCO version
Parts:
- R10, R11, R12, R13, R14, R15, R16: footprint Resistor_SMD:R_1206_3216Metric -> Resistor_SMD:R_2512_6332Metric
Changed lines of the file:
@@
 F 0 "R16" H 3659 8746 50  0000 L CNN
 F 1 "30" H 3659 8655 50  0000 L CNN
-F 2 "Resistor_SMD:R_1206_3216Metric" H 3600 8700 50  0001 C CNN
+F 2 "Resistor_SMD:R_2512_6332Metric" H 3600 8700 50  0001 C CNN
 F 3 "~" H 3600 8700 50  0001 C CNN
 	1    3600 8700
@@
 F 0 "R15" H 3659 7696 50  0000 L CNN
 F 1 "30" H 3659 7605 50  0000 L CNN
-F 2 "Resistor_SMD:R_1206_3216Metric" H 3600 7650 50  0001 C CNN
+F 2 "Resistor_SMD:R_2512_6332Metric" H 3600 7650 50  0001 C CNN
 F 3 "~" H 3600 7650 50  0001 C CNN
 	1    3600 7650
@@
 F 0 "R14" H 3659 6646 50  0000 L CNN
 F 1 "30" H 3659 6555 50  0000 L CNN
-F 2 "Resistor_SMD:R_1206_3216Metric" H 3600 6600 50  0001 C CNN
+F 2 "Resistor_SMD:R_2512_6332Metric" H 3600 6600 50  0001 C CNN
 F 3 "~" H 3600 6600 50  0001 C CNN
 	1    3600 6600
@@
 F 0 "R13" H 3659 5596 50  0000 L CNN
 F 1 "30" H 3659 5505 50  0000 L CNN
-F 2 "Resistor_SMD:R_1206_3216Metric" H 3600 5550 50  0001 C CNN
+F 2 "Resistor_SMD:R_2512_6332Metric" H 3600 5550 50  0001 C CNN
 F 3 "~" H 3600 5550 50  0001 C CNN
 	1    3600 5550
@@
 F 0 "R12" H 3659 4546 50  0000 L CNN
 F 1 "30" H 3659 4455 50  0000 L CNN
-F 2 "Resistor_SMD:R_1206_3216Metric" H 3600 4500 50  0001 C CNN
+F 2 "Resistor_SMD:R_2512_6332Metric" H 3600 4500 50  0001 C CNN
 F 3 "~" H 3600 4500 50  0001 C CNN
 	1    3600 4500
@@
 F 0 "R11" H 3659 3496 50  0000 L CNN
 F 1 "30" H 3659 3405 50  0000 L CNN
-F 2 "Resistor_SMD:R_1206_3216Metric" H 3600 3450 50  0001 C CNN
+F 2 "Resistor_SMD:R_2512_6332Metric" H 3600 3450 50  0001 C CNN
 F 3 "~" H 3600 3450 50  0001 C CNN
 	1    3600 3450
@@
 F 0 "R10" H 3659 2446 50  0000 L CNN
 F 1 "30" H 3659 2355 50  0000 L CNN
-F 2 "Resistor_SMD:R_1206_3216Metric" H 3600 2400 50  0001 C CNN
+F 2 "Resistor_SMD:R_2512_6332Metric" H 3600 2400 50  0001 C CNN
 F 3 "~" H 3600 2400 50  0001 C CNN
 	1    3600 2400
