File: Hardware/bmsLV.kicad_pcb (KiCad board)
At the start: 2 copper layers, 45 parts, among them J1 Conn_01x06_Male, J2 Conn_01x03_Female, J3 Conn_01x03_Female, J4 Conn_01x02_Female, J5 Conn_01x02_Female, SW1 SW_Push, U1 STM32F103C8Tx, U2 LM1117-3.3, U3 LM1117-3.3, U4 LM1117-3.3, U5 LM2596S-5, U6 MCP2562-H-SN, Y1 Crystal

Commit message: Save before ZCO version
Parts:
- removed U5: LM2596S-5, Package_TO_SOT_SMD:TO-263-5_TabPin3
- removed U6: MCP2562-H-SN, Package_SO:SOIC-8_3.9x4.9mm_P1.27mm
- added C20: 10nF, Capacitor_SMD:C_1206_3216Metric, F.Cu at (210.8, 58.6)
- added C21: 10nF, Capacitor_SMD:C_1206_3216Metric, F.Cu at (173.5, 85.5)
- added C22: 10nF, Capacitor_SMD:C_1206_3216Metric, F.Cu at (202.5, 67.4)
- added C23: 10nF, Capacitor_SMD:C_1206_3216Metric, F.Cu at (217.2, 53.0)
- added C24: 10nF, Capacitor_SMD:C_1206_3216Metric, F.Cu at (185.0, 82.2)
- added C25: 1u, Capacitor_SMD:C_1206_3216Metric, F.Cu at (202.5, 64.1)
- added C26: 1u, Capacitor_SMD:C_1206_3216Metric, F.Cu at (179.1, 85.5)
- added C27: 1u, Capacitor_SMD:C_1206_3216Metric, F.Cu at (184.7, 85.5)
- added C28: 1u, Capacitor_SMD:C_1206_3216Metric, F.Cu at (179.4, 82.2)
- added C29: 0.1u, Capacitor_SMD:C_0603_1608Metric, F.Cu at (195.1, 87.2)
- added C30: 100n, Capacitor_SMD:C_1206_3216Metric, F.Cu at (253.8, 99.9)
- added C31: 100n, Capacitor_SMD:C_1206_3216Metric, F.Cu at (253.8, 96.6)
- added C32: 100n, Capacitor_SMD:C_1206_3216Metric, F.Cu at (236.0, 111.4)
- added C33: 100n, Capacitor_SMD:C_1206_3216Metric, F.Cu at (253.8, 93.3)
- added C34: 100n, Capacitor_SMD:C_1206_3216Metric, F.Cu at (230.4, 111.4)
- added C35: 100n, Capacitor_SMD:C_1206_3216Metric, F.Cu at (219.1, 111.4)
- added D10: 9.1V, Diode_SMD:D_SMB, F.Cu at (189.1, 72.2)
- added D11: 9.1V, Diode_SMD:D_SMB, F.Cu at (201.9, 54.1)
- added D12: 9.1V, Diode_SMD:D_SMB, F.Cu at (180.8, 77.8)
- added D13: 9.1V, Diode_SMD:D_SMB, F.Cu at (189.1, 77.8)
- added D14: 9.1V, Diode_SMD:D_SMB, F.Cu at (180.8, 72.2)
- added D15: 9.1V, Diode_SMD:D_SMB, F.Cu at (210.2, 54.1)
- added D16: Prostownicza, Diode_SMD:D_SMB, F.Cu at (130.4, 69.8)
- added D5: D_Schottky, Diode_SMD:D_SMB, F.Cu at (36.4, 109.9)
- added D6: D_Schottky, Diode_SMD:D_SMB, F.Cu at (78.3, 106.0)
- added D7: D_Schottky, Diode_SMD:D_SMB, F.Cu at (44.2, 114.9)
- added D8: D_TVS_x2_AAC, Package_TO_SOT_SMD:SOT-23, F.Cu at (159.3, 118.7)
- added D9: 9.1V, Diode_SMD:D_SMB, F.Cu at (203.9, 59.7)
- added FB1: Ferrite_Bead_Small, Capacitor_SMD:C_1206_3216Metric, F.Cu at (36.7, 106.0)
- added J10: Conn_01x01_Female, CellPad:CellPad, F.Cu at (48.2, 62.2)
- added J11: Conn_01x01_Female, CellPad:CellPad, F.Cu at (27.9, 62.2)
- added J12: Conn_01x01_Female, CellPad:CellPad, F.Cu at (28.1, 112.7)
- added J13: Conn_01x04_Male, Connector_PinHeader_2.54mm:PinHeader_1x04_P2.54mm_Vertical, F.Cu at (122.6, 109.9)
- added J6: Conn_01x01_Female, CellPad:CellPad, F.Cu at (129.1, 62.2)
- added J7: Conn_01x01_Female, CellPad:CellPad, F.Cu at (108.9, 62.2)
- added J8: Conn_01x01_Female, CellPad:CellPad, F.Cu at (88.7, 62.2)
- added J9: Conn_01x01_Female, CellPad:CellPad, F.Cu at (68.4, 62.2)
- added K1: RM85V7, RM85V7:RM85V7, F.Cu at (130.2, 92.7)
- added LTC1: LTC6810-1, Package_SO:SSOP-44_5.3x12.8mm_P0.5mm, F.Cu at (171.2, 58.5)
- added Q1: BSS138, Package_TO_SOT_SMD:SOT-23, F.Cu at (124.2, 69.5)
- added Q2: Q_PMOS_GSD, Package_TO_SOT_SMD:SOT-23W, F.Cu at (212.6, 72.3)
- added Q3: Q_PMOS_GSD, Package_TO_SOT_SMD:SOT-23W, F.Cu at (219.0, 63.5)
- added Q4: Q_PMOS_GSD, Package_TO_SOT_SMD:SOT-23W, F.Cu at (228.1, 56.9)
- added Q5: Q_PMOS_GSD, Package_TO_SOT_SMD:SOT-23W, F.Cu at (201.5, 84.9)
- added Q6: Q_PMOS_GSD, Package_TO_SOT_SMD:SOT-23W, F.Cu at (223.9, 63.5)
- added Q7: Q_PMOS_GSD, Package_TO_SOT_SMD:SOT-23W, F.Cu at (207.1, 78.9)
- added Q8: Q_PMOS_GSD, Package_TO_SOT_SMD:SOT-23W, F.Cu at (212.6, 76.9)
- added Q9: Q_NPN_BCE, Package_TO_SOT_SMD:SOT-23W, F.Cu at (219.0, 68.0)
- added R10: 30, Resistor_SMD:R_2512_6332Metric, F.Cu at (228.4, 53.0)
- added R11: 30, Resistor_SMD:R_2512_6332Metric, F.Cu at (196.1, 71.1)
- added R12: 30, Resistor_SMD:R_2512_6332Metric, F.Cu at (167.8, 85.5)
- added R13: 30, Resistor_SMD:R_2512_6332Metric, F.Cu at (201.7, 71.1)
- added R14: 30, Resistor_SMD:R_2512_6332Metric, F.Cu at (207.3, 75.0)
- added R15: 30, Resistor_SMD:R_2512_6332Metric, F.Cu at (201.8, 81.0)
- added R16: 30, Resistor_SMD:R_2512_6332Metric, F.Cu at (213.7, 68.4)
- added R17: 1k, Resistor_SMD:R_1206_3216Metric, F.Cu at (222.1, 59.6)
- added R18: 1k, Resistor_SMD:R_1206_3216Metric, F.Cu at (201.7, 77.7)
- added R19: 1k, Resistor_SMD:R_1206_3216Metric, F.Cu at (207.3, 71.7)
- added R20: 1k, Resistor_SMD:R_1206_3216Metric, F.Cu at (196.2, 84.3)
- added R21: 1k, Resistor_SMD:R_1206_3216Metric, F.Cu at (190.6, 82.2)
- added R22: 1k, Resistor_SMD:R_1206_3216Metric, F.Cu at (213.7, 65.1)
- added R23: 1k, Resistor_SMD:R_1206_3216Metric, F.Cu at (222.8, 56.3)
- added R24: 100, Resistor_SMD:R_1206_3216Metric, F.Cu at (196.2, 81.0)
- added R25: 100, Resistor_SMD:R_1206_3216Metric, F.Cu at (208.1, 68.4)
- added R26: 100, Resistor_SMD:R_1206_3216Metric, F.Cu at (216.5, 59.6)
- added R27: 100, Resistor_SMD:R_1206_3216Metric, F.Cu at (201.7, 74.4)
- added R28: 100, Resistor_SMD:R_1206_3216Metric, F.Cu at (208.1, 65.1)
- added R29: 100, Resistor_SMD:R_1206_3216Metric, F.Cu at (190.3, 85.5)
- added R30: 100, Resistor_SMD:R_1206_3216Metric, F.Cu at (196.1, 77.7)
- added R31: 100, Resistor_SMD:R_1206_3216Metric, F.Cu at (222.8, 53.0)
- added R32: 100, Resistor_SMD:R_1206_3216Metric, F.Cu at (217.2, 56.3)
- added R33: 10K, Resistor_SMD:R_1206_3216Metric, F.Cu at (224.7, 111.4)
- added R34: 10K, Resistor_SMD:R_1206_3216Metric, F.Cu at (241.6, 111.4)
- added R35: 10K, Resistor_SMD:R_1206_3216Metric, F.Cu at (253.8, 103.2)
- added R36: 10K, Resistor_SMD:R_1206_3216Metric, F.Cu at (247.2, 111.4)
- added R37: 10K, Resistor_SMD:R_1206_3216Metric, F.Cu at (253.8, 106.5)
- added R38: 10K, Resistor_SMD:R_1206_3216Metric, F.Cu at (252.8, 111.4)
- added R7: 100, Resistor_SMD:R_1206_3216Metric, F.Cu at (118.7, 70.0)
- added R8: 10K, Resistor_SMD:R_1206_3216Metric, F.Cu at (121.3, 70.0)
- added R9: 120, Resistor_SMD:R_1206_3216Metric, F.Cu at (170.2, 114.9)
- added TH1: Thermistor_PTC, Connector_PinHeader_2.54mm:PinHeader_1x02_P2.54mm_Vertical, F.Cu at (242.7, 105.2)
- added TH2: Thermistor_PTC, Connector_PinHeader_2.54mm:PinHeader_1x02_P2.54mm_Vertical, F.Cu at (242.7, 96.2)
- added TH3: Thermistor_PTC, Connector_PinHeader_2.54mm:PinHeader_1x02_P2.54mm_Vertical, F.Cu at (231.1, 105.2)
- added TH4: Thermistor_PTC, Connector_PinHeader_2.54mm:PinHeader_1x02_P2.54mm_Vertical, F.Cu at (231.1, 96.2)
- added TH5: Thermistor_PTC, Connector_PinHeader_2.54mm:PinHeader_1x02_P2.54mm_Vertical, F.Cu at (219.6, 105.2)
- added TH6: Thermistor_PTC, Connector_PinHeader_2.54mm:PinHeader_1x02_P2.54mm_Vertical, F.Cu at (219.6, 96.2)
- C1, C2: value C_Small -> 22p
- C10: value CP_Small -> 47n; footprint Capacitor_SMD:CP_Elec_6.3x7.7 -> Capacitor_SMD:C_1206_3216Metric
- C11: value C_Small -> 680u; footprint Capacitor_SMD:C_1206_3216Metric -> Capacitor_SMD:CP_Elec_6.3x7.7
- C12, C13, C14, C16, C3, C4, C5, C6, C7, C8: value C_Small -> 100n
- C15: value C_Small -> 220uF; footprint Capacitor_SMD:C_1206_3216Metric -> Capacitor_SMD:CP_Elec_6.3x7.7
- C17: value CP_Small -> 100n; footprint Capacitor_SMD:CP_Elec_6.3x7.7 -> Capacitor_SMD:C_1206_3216Metric
- C18, C19: value C_Small -> 10nF
- C9: value C_Small -> 330p
- D2, D3: value D_Schottky -> LED; footprint Diode_SMD:D_SMB -> LED_SMD:LED_1206_3216Metric
- D4: value D_TVS_x2_AAC -> LED; footprint Package_TO_SOT_SMD:SOT-23 -> LED_SMD:LED_1206_3216Metric
- J2: value Conn_01x03_Female -> USB_B_Mini; footprint TerminalBlock:TerminalBlock_bornier-3_P5.08mm -> Connector_USB:USB_Micro-B_Molex_47346-0001
- J3: value Conn_01x03_Female -> Conn_01x02_Female; footprint TerminalBlock:TerminalBlock_bornier-3_P5.08mm -> TerminalBlock:TerminalBlock_bornier-2_P5.08mm
- J4: value Conn_01x02_Female -> Conn_01x02_Male; footprint TerminalBlock:TerminalBlock_bornier-2_P5.08mm -> Connector_PinHeader_2.54mm:PinHeader_1x02_P2.54mm_Vertical
- L1: value L_Small -> 10u
- L2: value L_Small -> 33u
- R1, R2: value 100K -> 1K
- R3: value 500 -> 1K
- R4: value R_Small -> 1K
- R5: value R_Small -> 100K
- R6: value 120 -> 100K
- U3: value LM1117-3.3 -> LM2596S-5; footprint Package_TO_SOT_SMD:SOT-223 -> Package_TO_SOT_SMD:TO-263-5_TabPin3
- U4: value LM1117-3.3 -> MCP2562-H-SN; footprint Package_TO_SOT_SMD:SOT-223 -> Package_SO:SOIC-8_3.9x4.9mm_P1.27mm
- moved C18 124.8 mm to (210.8, 61.8)
- moved J3 115.7 mm to (33.0, 96.5), turned to 270 degrees
- moved C19 100.6 mm to (196.1, 74.4)
- moved F1 95.3 mm to (36.4, 114.9), turned to 180 degrees
- moved C16 91.1 mm to (177.2, 125.9), turned to 270 degrees
- moved SW1 90.3 mm to (93.3, 110.4)
- moved C6 88.7 mm to (100.2, 105.4), turned to 180 degrees
- moved L1 87.8 mm to (100.3, 108.0)
- moved C9 86.9 mm to (43.2, 106.0), turned to 180 degrees
- moved C12 83.4 mm to (43.0, 111.1), turned to 180 degrees
- moved Y1 81.2 mm to (94.6, 99.5), turned to 270 degrees
- moved J5 79.5 mm to (160.0, 128.9)
- moved U4 79.4 mm to (174.7, 120.7)
- moved R4 78.3 mm to (111.1, 114.4), turned to 270 degrees
- moved C1 77.7 mm to (99.1, 97.0), turned to 270 degrees
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Connections:
- C11 pad 1: +5V -> Net-(C10-Pad1)
- C12 pad 1: +5V -> Net-(C10-Pad1)
- C15 pad 1: +3.3VA -> +5VD
- C16 pad 1: +3.3VADC -> SW_VDD
- C18 pad 1: SW_VDD -> SW_GND
- C18 pad 2: SW_GND -> Net-(C18-Pad2)
- C19 pad 1: +5V -> SW_GND
- C19 pad 2: SW_GND -> Net-(C19-Pad2)
- C9 pad 1: Net-(C10-Pad1) -> Net-(C9-Pad1)
- D2 pad 1: Net-(C10-Pad1) -> Net-(D2-Pad1)
- D2 pad 2: SW_GND -> Net-(D2-Pad2)
- D3 pad 2: SW_GND -> Net-(D3-Pad2)
- D4 pad 1: CANL -> Net-(D4-Pad1)
- D4 pad 2: CANH -> Net-(D4-Pad2)
- F1 pad 1: Net-(C10-Pad1) -> Net-(C9-Pad1)
- F1 pad 2: Net-(F1-Pad2) -> VCC
- J2 pad 1: Net-(J2-Pad1) -> +5V
- J2 pad 2: Ain0 -> USB_DM
- J2 pad 3: SW_GND -> USB_DP
- J3 pad 1: +3.3VADC -> SW_GND
- J3 pad 2: Ain1 -> VCC
- J4 pad 1: SW_GND -> CANL
- J4 pad 2: Net-(F1-Pad2) -> Net-(J4-Pad2)
- L2 pad 1: Net-(D3-Pad1) -> Net-(D7-Pad1)
- L2 pad 2: +5V -> +5VD
- R1 pad 1: SW_VDD -> Net-(D1-Pad2)
- R1 pad 2: SW_NRST -> SW_VDD
- R2 pad 1: Net-(R2-Pad1) -> Net-(D2-Pad2)
- R2 pad 2: SW_GND -> SW_VDD
- R3 pad 1: SW_VDD -> Net-(D3-Pad2)
- R3 pad 2: Net-(D1-Pad2) -> SW_VDD
- R4 pad 1: +3.3VA -> Net-(D4-Pad2)
- R4 pad 2: Net-(J2-Pad1) -> SW_VDD
- R5 pad 1: Net-(J3-Pad3) -> SW_VDD
- R5 pad 2: SW_GND -> SW_NRST
- R6 pad 1: CANH -> Net-(R6-Pad1)
- R6 pad 2: CANL -> SW_GND
- U1 pad 10: Ain0 -> Net-(U1-Pad10)
- U1 pad 11: Ain1 -> Net-(U1-Pad11)
- U1 pad 12: Net-(U1-Pad12) -> En_Relay
- U1 pad 13: Net-(U1-Pad13) -> Term_1
- U1 pad 14: Net-(U1-Pad14) -> Term_2
- U1 pad 15: Net-(D1-Pad1) -> Term_3
- U1 pad 16: Net-(U1-Pad16) -> Term_4
- U1 pad 17: Net-(U1-Pad17) -> Term_5
- U1 pad 18: Net-(U1-Pad18) -> Term_6
- U1 pad 19: Net-(U1-Pad19) -> Net-(D1-Pad1)
- U1 pad 20: Net-(U1-Pad20) -> Net-(D2-Pad1)
- U1 pad 21: Net-(U1-Pad21) -> Net-(D3-Pad1)
- U1 pad 22: Net-(U1-Pad22) -> Net-(D4-Pad1)
- U1 pad 32: RX_Can -> USB_DM
- U1 pad 33: TX_Can -> USB_DP
- U1 pad 38: Net-(U1-Pad38) -> CS
- U1 pad 39: Net-(U1-Pad39) -> SCK
- U1 pad 40: Net-(U1-Pad40) -> MISO
- U1 pad 41: Net-(U1-Pad41) -> MOSI
- U1 pad 44: Net-(R2-Pad1) -> Net-(R6-Pad1)
- U1 pad 45: Net-(U1-Pad45) -> RX_Can
- U1 pad 46: Net-(U1-Pad46) -> TX_Can
- U3 pad 1: SW_GND -> Net-(C10-Pad1)
- U3 pad 2: +3.3VA -> Net-(D7-Pad1)
- U3 pad 3: +5V -> SW_GND
- U3 pad 4: (no net) -> +5VD
- U4 pad 1: SW_GND -> TX_Can
- U4 pad 2: +3.3VADC -> SW_GND
- U4 pad 4: (no net) -> RX_Can
Other:
- board outline added: 121.2 x 60.6 mm

Commit message: ZCO version
Parts:
- moved TH1 127.8 mm to (117.0, 82.4), turned to 90 degrees
- moved TH2 126.9 mm to (117.0, 78.8), turned to 90 degrees
- moved TH3 119.1 mm to (116.9, 71.3), turned to 90 degrees
- moved TH4 118.8 mm to (116.9, 63.7), turned to 90 degrees
- moved TH5 107.0 mm to (116.9, 75.1), turned to 90 degrees
- moved TH6 106.6 mm to (116.9, 67.5), turned to 90 degrees
- moved R16 98.4 mm to (118.0, 91.2), turned to 90 degrees
- moved C1 95.4 mm to (194.1, 88.5)
- moved C2 95.4 mm to (194.1, 93.2)
- moved C4 95.4 mm to (194.1, 83.7)
- moved C5 95.4 mm to (196.6, 83.7)
- moved D1 95.4 mm to (198.5, 101.2)
- moved D16 95.4 mm to (225.4, 61.3)
- moved D4 95.4 mm to (206.1, 101.2)
- moved D5 95.4 mm to (131.4, 101.3)
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Other:
- outline, holes or cut-outs redrawn
