File: Hardware/power.sch (KiCad schematic (older format))
At the start: 15 parts, among them U2 LM1117-3.3, U3 LM2596S-5

Commit message: Some changes
Parts:
- U3: symbol Regulator_Switching:LM2596S-5 -> bmsLV-rescue:LM2596S-5-Regulator_Switching
Changed lines of the file:
@@
 EESchema Schematic File Version 4
-EELAYER 30 0
+LIBS:bmsLV-cache
+EELAYER 29 0
 EELAYER END
 $Descr A4 11693 8268
@@
 $EndDescr
 $Comp
-L Regulator_Switching:LM2596S-5 U3
+L bmsLV-rescue:LM2596S-5-Regulator_Switching U3
 U 1 1 5FADABDE
 P 3450 2250

Commit message: footprint update
Parts:
- U2: footprint Package_TO_SOT_SMD:SOT-223 -> Package_TO_SOT_SMD:SOT-223-3_TabPin2
Changed lines of the file:
@@
 EESchema Schematic File Version 4
-LIBS:bmsLV-cache
-EELAYER 29 0
+EELAYER 30 0
 EELAYER END
 $Descr A4 11693 8268
@@
 F 0 "U2" H 3400 3942 50  0000 C CNN
 F 1 "LM1117-3.3" H 3400 3851 50  0000 C CNN
-F 2 "Package_TO_SOT_SMD:SOT-223" H 3400 3700 50  0001 C CNN
+F 2 "Package_TO_SOT_SMD:SOT-223-3_TabPin2" H 3400 3700 50  0001 C CNN
 F 3 "http://www.ti.com/lit/ds/symlink/lm1117.pdf" H 3400 3700 50  0001 C CNN
 	1    3400 3700
