File: Hardware/power.sch (KiCad schematic (older format))
At the start: 15 parts, among them U2 LM1117-3.3, U3 LM2596S-5

Commit message: Software update 3
Current sensor added to PCB (through wires)
Current sensor handling added
Cell balance working! (HUGE PART OF UPDATE)
CheckError function modified (a lot of more error added)
Serial print function added (not tested)
+ some cosmetic changes
Parts:
- C10, C12, C13, C14, C9: symbol Device:C_Small -> bmsLV-rescue:C_Small-Device
- C11, C15: symbol Device:CP_Small -> bmsLV-rescue:CP_Small-Device
- D5, D6, D7: symbol Device:D_Schottky -> bmsLV-rescue:D_Schottky-Device
- F1: symbol Device:Fuse -> bmsLV-rescue:Fuse-Device
- FB1: symbol Device:Ferrite_Bead_Small -> bmsLV-rescue:Ferrite_Bead_Small-Device
- L2: symbol Device:L_Small -> bmsLV-rescue:L_Small-Device
- U2: symbol Regulator_Linear:LM1117-3.3 -> bmsLV-rescue:LM1117-3.3-Regulator_Linear
Changed lines of the file:
@@
 $EndComp
 $Comp
-L Device:C_Small C12
+L bmsLV-rescue:C_Small-Device C12
 U 1 1 5FADDCE9
 P 2800 2500
@@
 $EndComp
 $Comp
-L Device:L_Small L2
+L bmsLV-rescue:L_Small-Device L2
 U 1 1 5FADEE69
 P 4650 2350
@@
 $EndComp
 $Comp
-L Device:CP_Small C11
+L bmsLV-rescue:CP_Small-Device C11
 U 1 1 5FAE0A9C
 P 2600 2500
@@
 $EndComp
 $Comp
-L Device:CP_Small C15
+L bmsLV-rescue:CP_Small-Device C15
 U 1 1 5FAE3D09
 P 5000 2450
@@
 $EndComp
 $Comp
-L Device:D_Schottky D7
+L bmsLV-rescue:D_Schottky-Device D7
 U 1 1 5FAE479F
 P 4250 2500
@@
 	3450 2850 3450 2950
 $Comp
-L power:GND #PWR025
+L bmsLV-rescue:GND-power #PWR025
 U 1 1 5FAED334
 P 3450 2950
@@
 $EndComp
 $Comp
-L Device:Fuse F1
+L bmsLV-rescue:Fuse-Device F1
 U 1 1 5FAEFFDF
 P 1350 2150
@@
 	1500 2150 1550 2150
 $Comp
-L Device:D_Schottky D5
+L bmsLV-rescue:D_Schottky-Device D5
 U 1 1 5FAF1827
 P 1550 2300
@@
 	1550 2450 1550 2850
 $Comp
-L Regulator_Linear:LM1117-3.3 U2
+L bmsLV-rescue:LM1117-3.3-Regulator_Linear U2
 U 1 1 5FAF5A27
 P 3400 3700
@@
 $EndComp
 $Comp
-L Device:C_Small C13
+L bmsLV-rescue:C_Small-Device C13
 U 1 1 5FAF6BC0
 P 2800 3800
@@
 $EndComp
 $Comp
-L Device:C_Small C14
+L bmsLV-rescue:C_Small-Device C14
 U 1 1 5FAF733B
 P 4000 3800
@@
 	3400 4000 3400 4050
 $Comp
-L power:GND #PWR024
+L bmsLV-rescue:GND-power #PWR024
 U 1 1 5FAFB775
 P 3400 4050
@@
 $EndComp
 $Comp
-L power:+5V #PWR023
+L bmsLV-rescue:+5V-power #PWR023
 U 1 1 5FAFC4B2
 P 2650 3650
@@
 $EndComp
 $Comp
-L power:+3.3V #PWR026
+L bmsLV-rescue:+3.3V-power #PWR026
 U 1 1 5FAFCB57
 P 4250 3550
@@
 $EndComp
 $Comp
-L Device:D_Schottky D6
+L bmsLV-rescue:D_Schottky-Device D6
 U 1 1 5FFC9BA8
 P 2400 3700
@@
 $EndComp
 $Comp
-L power:+5VD #PWR027
+L bmsLV-rescue:+5VD-power #PWR027
 U 1 1 5FFCAC1E
 P 5800 2350
@@
 	2150 3700 2150 3650
 $Comp
-L power:+5VD #PWR022
+L bmsLV-rescue:+5VD-power #PWR022
 U 1 1 5FFCC30E
 P 2150 3650
@@
 	2650 3700 2800 3700
 $Comp
-L Device:C_Small C9
+L bmsLV-rescue:C_Small-Device C9
 U 1 1 5FFCD640
 P 1950 2500
@@
 $EndComp
 $Comp
-L Device:C_Small C10
+L bmsLV-rescue:C_Small-Device C10
 U 1 1 5FFCE3B8
 P 2300 2500
@@
 $EndComp
 $Comp
-L Device:Ferrite_Bead_Small FB1
+L bmsLV-rescue:Ferrite_Bead_Small-Device FB1
 U 1 1 5FFCEC0C
 P 2150 2150
@@
 	2800 2850 2950 2850
 $Comp
-L power:VCC #PWR0103
+L bmsLV-rescue:VCC-power #PWR0103
 U 1 1 5FFFB3C9
 P 1050 2150
