File: Hardware/Thermistors.sch (KiCad schematic (older format))
At the start: 18 parts

Commit message: Power update
Parts:
- renumbered C28 to C30, C29 to C31, C30 to C32, C31 to C33, C32 to C34, C33 to C35
Changed lines of the file:
@@
 	4850 3500 4850 3600
 $Comp
-L Device:C_Small C28
+L Device:C_Small C30
 U 1 1 606327DA
 P 4850 3700
-F 0 "C28" H 4942 3746 50  0000 L CNN
+F 0 "C30" H 4942 3746 50  0000 L CNN
 F 1 "100n" H 4942 3655 50  0000 L CNN
 F 2 "Capacitor_SMD:C_1206_3216Metric" H 4850 3700 50  0001 C CNN
@@
 $EndComp
 $Comp
-L Device:C_Small C29
+L Device:C_Small C31
 U 1 1 6063CCC6
 P 5150 3700
-F 0 "C29" H 5242 3746 50  0000 L CNN
+F 0 "C31" H 5242 3746 50  0000 L CNN
 F 1 "100n" H 5242 3655 50  0000 L CNN
 F 2 "Capacitor_SMD:C_1206_3216Metric" H 5150 3700 50  0001 C CNN
@@
 	5150 3200 5150 3600
 $Comp
-L Device:C_Small C30
+L Device:C_Small C32
 U 1 1 6063DBA9
 P 5450 3700
-F 0 "C30" H 5542 3746 50  0000 L CNN
+F 0 "C32" H 5542 3746 50  0000 L CNN
 F 1 "100n" H 5542 3655 50  0000 L CNN
 F 2 "Capacitor_SMD:C_1206_3216Metric" H 5450 3700 50  0001 C CNN
@@
 	5450 2900 5450 3600
 $Comp
-L Device:C_Small C31
+L Device:C_Small C33
 U 1 1 6063E87B
 P 5750 3700
-F 0 "C31" H 5842 3746 50  0000 L CNN
+F 0 "C33" H 5842 3746 50  0000 L CNN
 F 1 "100n" H 5842 3655 50  0000 L CNN
 F 2 "Capacitor_SMD:C_1206_3216Metric" H 5750 3700 50  0001 C CNN
@@
 	5750 2600 5750 3600
 $Comp
-L Device:C_Small C32
+L Device:C_Small C34
 U 1 1 6063F5AA
 P 6050 3700
-F 0 "C32" H 6142 3746 50  0000 L CNN
+F 0 "C34" H 6142 3746 50  0000 L CNN
 F 1 "100n" H 6142 3655 50  0000 L CNN
 F 2 "Capacitor_SMD:C_1206_3216Metric" H 6050 3700 50  0001 C CNN
@@
 	6050 2300 6050 3600
 $Comp
-L Device:C_Small C33
+L Device:C_Small C35
 U 1 1 60640F90
 P 6350 3700
-F 0 "C33" H 6442 3746 50  0000 L CNN
+F 0 "C35" H 6442 3746 50  0000 L CNN
 F 1 "100n" H 6442 3655 50  0000 L CNN
 F 2 "Capacitor_SMD:C_1206_3216Metric" H 6350 3700 50  0001 C CNN

Commit message: pcb layout nearly done
Parts:
- TH1, TH2, TH3, TH4, TH5, TH6: footprint TerminalBlock:TerminalBlock_bornier-2_P5.08mm -> Connector_PinHeader_2.54mm:PinHeader_1x02_P2.54mm_Vertical
Changed lines of the file:
@@
 EESchema Schematic File Version 4
+LIBS:bmsLV-cache
 EELAYER 30 0
 EELAYER END
@@
 F 0 "TH1" V 2885 3800 50  0000 C CNN
 F 1 "Thermistor_PTC" V 2794 3800 50  0000 C CNN
-F 2 "TerminalBlock:TerminalBlock_bornier-2_P5.08mm" H 2700 3600 50  0001 L CNN
+F 2 "Connector_PinHeader_2.54mm:PinHeader_1x02_P2.54mm_Vertical" H 2700 3600 50  0001 L CNN
 F 3 "~" H 2650 3800 50  0001 C CNN
 	1    2650 3800
@@
 F 0 "TH2" V 3285 3800 50  0000 C CNN
 F 1 "Thermistor_PTC" V 3194 3800 50  0000 C CNN
-F 2 "TerminalBlock:TerminalBlock_bornier-2_P5.08mm" H 3100 3600 50  0001 L CNN
+F 2 "Connector_PinHeader_2.54mm:PinHeader_1x02_P2.54mm_Vertical" H 3100 3600 50  0001 L CNN
 F 3 "~" H 3050 3800 50  0001 C CNN
 	1    3050 3800
@@
 F 0 "TH3" V 3685 3800 50  0000 C CNN
 F 1 "Thermistor_PTC" V 3594 3800 50  0000 C CNN
-F 2 "TerminalBlock:TerminalBlock_bornier-2_P5.08mm" H 3500 3600 50  0001 L CNN
+F 2 "Connector_PinHeader_2.54mm:PinHeader_1x02_P2.54mm_Vertical" H 3500 3600 50  0001 L CNN
 F 3 "~" H 3450 3800 50  0001 C CNN
 	1    3450 3800
@@
 F 0 "TH4" V 4085 3800 50  0000 C CNN
 F 1 "Thermistor_PTC" V 3994 3800 50  0000 C CNN
-F 2 "TerminalBlock:TerminalBlock_bornier-2_P5.08mm" H 3900 3600 50  0001 L CNN
+F 2 "Connector_PinHeader_2.54mm:PinHeader_1x02_P2.54mm_Vertical" H 3900 3600 50  0001 L CNN
 F 3 "~" H 3850 3800 50  0001 C CNN
 	1    3850 3800
@@
 F 0 "TH5" V 4485 3800 50  0000 C CNN
 F 1 "Thermistor_PTC" V 4394 3800 50  0000 C CNN
-F 2 "TerminalBlock:TerminalBlock_bornier-2_P5.08mm" H 4300 3600 50  0001 L CNN
+F 2 "Connector_PinHeader_2.54mm:PinHeader_1x02_P2.54mm_Vertical" H 4300 3600 50  0001 L CNN
 F 3 "~" H 4250 3800 50  0001 C CNN
 	1    4250 3800
@@
 F 0 "TH6" V 4885 3800 50  0000 C CNN
 F 1 "Thermistor_PTC" V 4794 3800 50  0000 C CNN
-F 2 "TerminalBlock:TerminalBlock_bornier-2_P5.08mm" H 4700 3600 50  0001 L CNN
+F 2 "Connector_PinHeader_2.54mm:PinHeader_1x02_P2.54mm_Vertical" H 4700 3600 50  0001 L CNN
 F 3 "~" H 4650 3800 50  0001 C CNN
 	1    4650 3800
