File: Hardware/Thermistors.sch (KiCad schematic (older format))
At the start: 18 parts

Commit message: Software update 3
Current sensor added to PCB (through wires)
Current sensor handling added
Cell balance working! (HUGE PART OF UPDATE)
CheckError function modified (a lot of more error added)
Serial print function added (not tested)
+ some cosmetic changes
Parts:
- C30, C31, C32, C33, C34, C35: symbol Device:C_Small -> bmsLV-rescue:C_Small-Device
- R33, R34, R35, R36, R37, R38: symbol Device:R_Small -> bmsLV-rescue:R_Small-Device
- TH1, TH2, TH3, TH4, TH5, TH6: symbol Device:Thermistor_PTC -> bmsLV-rescue:Thermistor_PTC-Device
Changed lines of the file:
@@
 	2000 2000 2350 2000
 $Comp
-L Device:R_Small R33
+L bmsLV-rescue:R_Small-Device R33
 U 1 1 6061BF07
 P 2450 2000
@@
 	2000 2300 2350 2300
 $Comp
-L Device:R_Small R34
+L bmsLV-rescue:R_Small-Device R34
 U 1 1 6061E665
 P 2450 2300
@@
 	2000 2600 2350 2600
 $Comp
-L Device:R_Small R35
+L bmsLV-rescue:R_Small-Device R35
 U 1 1 606208B8
 P 2450 2600
@@
 	2000 2900 2350 2900
 $Comp
-L Device:R_Small R36
+L bmsLV-rescue:R_Small-Device R36
 U 1 1 60621BF1
 P 2450 2900
@@
 	2000 3200 2350 3200
 $Comp
-L Device:R_Small R37
+L bmsLV-rescue:R_Small-Device R37
 U 1 1 6062228C
 P 2450 3200
@@
 	2000 3500 2350 3500
 $Comp
-L Device:R_Small R38
+L bmsLV-rescue:R_Small-Device R38
 U 1 1 60622889
 P 2450 3500
@@
 Connection ~ 2650 2000
 $Comp
-L Device:Thermistor_PTC TH1
+L bmsLV-rescue:Thermistor_PTC-Device TH1
 U 1 1 606242F5
 P 2650 3800
@@
 $EndComp
 $Comp
-L Device:Thermistor_PTC TH2
+L bmsLV-rescue:Thermistor_PTC-Device TH2
 U 1 1 60626217
 P 3050 3800
@@
 $EndComp
 $Comp
-L Device:Thermistor_PTC TH3
+L bmsLV-rescue:Thermistor_PTC-Device TH3
 U 1 1 606266F5
 P 3450 3800
@@
 $EndComp
 $Comp
-L Device:Thermistor_PTC TH4
+L bmsLV-rescue:Thermistor_PTC-Device TH4
 U 1 1 6062692C
 P 3850 3800
@@
 $EndComp
 $Comp
-L Device:Thermistor_PTC TH5
+L bmsLV-rescue:Thermistor_PTC-Device TH5
 U 1 1 60626CD3
 P 4250 3800
@@
 $EndComp
 $Comp
-L Device:Thermistor_PTC TH6
+L bmsLV-rescue:Thermistor_PTC-Device TH6
 U 1 1 60627523
 P 4650 3800
@@
 	3650 4100 3850 4100
 $Comp
-L power:GND #PWR058
+L bmsLV-rescue:GND-power #PWR058
 U 1 1 6062C049
 P 3650 4150
@@
 	4850 3500 4850 3600
 $Comp
-L Device:C_Small C30
+L bmsLV-rescue:C_Small-Device C30
 U 1 1 606327DA
 P 4850 3700
@@
 	4850 3800 4850 3850
 $Comp
-L power:GND #PWR059
+L bmsLV-rescue:GND-power #PWR059
 U 1 1 606341EE
 P 4850 3850
@@
 $EndComp
 $Comp
-L Device:C_Small C31
+L bmsLV-rescue:C_Small-Device C31
 U 1 1 6063CCC6
 P 5150 3700
@@
 	5150 3800 5150 3850
 $Comp
-L power:GND #PWR060
+L bmsLV-rescue:GND-power #PWR060
 U 1 1 6063CCCD
 P 5150 3850
@@
 	5150 3200 5150 3600
 $Comp
-L Device:C_Small C32
+L bmsLV-rescue:C_Small-Device C32
 U 1 1 6063DBA9
 P 5450 3700
@@
 	5450 3800 5450 3850
 $Comp
-L power:GND #PWR061
+L bmsLV-rescue:GND-power #PWR061
 U 1 1 6063DBB0
 P 5450 3850
@@
 	5450 2900 5450 3600
 $Comp
-L Device:C_Small C33
+L bmsLV-rescue:C_Small-Device C33
 U 1 1 6063E87B
 P 5750 3700
@@
 	5750 3800 5750 3850
 $Comp
-L power:GND #PWR062
+L bmsLV-rescue:GND-power #PWR062
 U 1 1 6063E882
 P 5750 3850
@@
 	5750 2600 5750 3600
 $Comp
-L Device:C_Small C34
+L bmsLV-rescue:C_Small-Device C34
 U 1 1 6063F5AA
 P 6050 3700
@@
 	6050 3800 6050 3850
 $Comp
-L power:GND #PWR063
+L bmsLV-rescue:GND-power #PWR063
 U 1 1 6063F5B1
 P 6050 3850
@@
 	6050 2300 6050 3600
 $Comp
-L Device:C_Small C35
+L bmsLV-rescue:C_Small-Device C35
 U 1 1 60640F90
 P 6350 3700
@@
 	6350 3800 6350 3850
 $Comp
-L power:GND #PWR064
+L bmsLV-rescue:GND-power #PWR064
 U 1 1 60640F97
 P 6350 3850
@@
 Term_6
 $Comp
-L power:+3.3V #PWR052
+L bmsLV-rescue:+3.3V-power #PWR052
 U 1 1 6064D34D
 P 2000 1950
@@
 $EndComp
 $Comp
-L power:+3.3V #PWR053
+L bmsLV-rescue:+3.3V-power #PWR053
 U 1 1 6064E1BD
 P 2000 2250
@@
 $EndComp
 $Comp
-L power:+3.3V #PWR054
+L bmsLV-rescue:+3.3V-power #PWR054
 U 1 1 6064EFA4
 P 2000 2550
@@
 $EndComp
 $Comp
-L power:+3.3V #PWR055
+L bmsLV-rescue:+3.3V-power #PWR055
 U 1 1 60650F26
 P 2000 2850
@@
 $EndComp
 $Comp
-L power:+3.3V #PWR056
+L bmsLV-rescue:+3.3V-power #PWR056
 U 1 1 60651C4E
 P 2000 3150
@@
 $EndComp
 $Comp
-L power:+3.3V #PWR057
+L bmsLV-rescue:+3.3V-power #PWR057
 U 1 1 60652A7D
 P 2000 3450
