File: Hardware/LTC.sch (KiCad schematic (older format))
At the start: 64 parts, among them J10 Conn_01x01_Female, J11 Conn_01x01_Female, J12 Conn_01x01_Female, J6 Conn_01x01_Female, J7 Conn_01x01_Female, J8 Conn_01x01_Female, J9 Conn_01x01_Female, Q2 Q_PMOS_GSD, Q3 Q_PMOS_GSD, Q4 Q_PMOS_GSD, Q5 Q_PMOS_GSD, Q6 Q_PMOS_GSD, Q7 Q_PMOS_GSD, Q8 Q_PMOS_GSD, Q9 Q_NPN_BCE

Commit message: Cosmetic changes in files
Parts:
- LTC1: symbol bms1-rescue:LTC6810-1-LTC6810-1 -> LTC6810-1:LTC6810-1-LTC6810-1
Changed lines of the file:
@@
 	8200 2600 8350 2600
 $Comp
-L bms1-rescue:LTC6810-1-LTC6810-1 LTC1
+L LTC6810-1:LTC6810-1-LTC6810-1 LTC1
 U 1 1 5FF8D74A
 P 7350 4100
+AR Path="/5FF8D74A" Ref="LTC1"  Part="1"
+AR Path="/5FF86554/5FF8D74A" Ref="LTC1"  Part="1"
 F 0 "LTC1" H 6450 6475 50  0000 C CNN
 F 1 "LTC6810-1" H 6450 6384 50  0000 C CNN

Commit message: Power update
Parts:
- C29: renamed from C27; footprint Capacitor_SMD:C_1206_3216Metric -> Capacitor_SMD:C_0603_1608Metric
- renumbered C16 to C18, C17 to C19, C18 to C20, C19 to C21, C20 to C22, C21 to C23, C22 to C24, C23 to C25, C24 to C26, C25 to C27, C26 to C28
Changed lines of the file:
@@
 	4050 8550 4250 8550
 $Comp
-L Device:C_Small C21
+L Device:C_Small C23
 U 1 1 601C6399
 P 4250 8650
-F 0 "C21" H 4158 8604 50  0000 R CNN
+F 0 "C23" H 4158 8604 50  0000 R CNN
 F 1 "10nF" H 4158 8695 50  0000 R CNN
 F 2 "Capacitor_SMD:C_1206_3216Metric" H 4250 8650 50  0001 C CNN
@@
 	4050 7500 4250 7500
 $Comp
-L Device:C_Small C20
+L Device:C_Small C22
 U 1 1 6011B7E6
 P 4250 7600
-F 0 "C20" H 4158 7554 50  0000 R CNN
+F 0 "C22" H 4158 7554 50  0000 R CNN
 F 1 "10nF" H 4158 7645 50  0000 R CNN
 F 2 "Capacitor_SMD:C_1206_3216Metric" H 4250 7600 50  0001 C CNN
@@
 	4050 6450 4250 6450
 $Comp
-L Device:C_Small C19
+L Device:C_Small C21
 U 1 1 601110FB
 P 4250 6550
-F 0 "C19" H 4158 6504 50  0000 R CNN
+F 0 "C21" H 4158 6504 50  0000 R CNN
 F 1 "10nF" H 4158 6595 50  0000 R CNN
 F 2 "Capacitor_SMD:C_1206_3216Metric" H 4250 6550 50  0001 C CNN
@@
 	4050 5400 4250 5400
 $Comp
-L Device:C_Small C18
+L Device:C_Small C20
 U 1 1 60106229
 P 4250 5500
-F 0 "C18" H 4158 5454 50  0000 R CNN
+F 0 "C20" H 4158 5454 50  0000 R CNN
 F 1 "10nF" H 4158 5545 50  0000 R CNN
 F 2 "Capacitor_SMD:C_1206_3216Metric" H 4250 5500 50  0001 C CNN
@@
 	4050 4350 4250 4350
 $Comp
-L Device:C_Small C17
+L Device:C_Small C19
 U 1 1 600FD81B
 P 4250 4450
-F 0 "C17" H 4158 4404 50  0000 R CNN
+F 0 "C19" H 4158 4404 50  0000 R CNN
 F 1 "10nF" H 4158 4495 50  0000 R CNN
 F 2 "Capacitor_SMD:C_1206_3216Metric" H 4250 4450 50  0001 C CNN
@@
 	4050 3300 4250 3300
 $Comp
-L Device:C_Small C16
+L Device:C_Small C18
 U 1 1 5FFBF39B
 P 4250 3400
-F 0 "C16" H 4158 3354 50  0000 R CNN
+F 0 "C18" H 4158 3354 50  0000 R CNN
 F 1 "10nF" H 4158 3445 50  0000 R CNN
 F 2 "Capacitor_SMD:C_1206_3216Metric" H 4250 3400 50  0001 C CNN
@@
 $EndComp
 $Comp
-L Device:C_Small C22
+L Device:C_Small C24
 U 1 1 5FF93E07
 P 4450 2350
-F 0 "C22" H 4358 2304 50  0000 R CNN
+F 0 "C24" H 4358 2304 50  0000 R CNN
 F 1 "10nF" H 4358 2395 50  0000 R CNN
 F 2 "Capacitor_SMD:C_1206_3216Metric" H 4450 2350 50  0001 C CNN
@@
 	7500 3250 7500 3300
 $Comp
-L Device:C_Small C25
+L Device:C_Small C27
 U 1 1 6019F5F8
 P 7500 3400
-F 0 "C25" H 7592 3446 50  0000 L CNN
+F 0 "C27" H 7592 3446 50  0000 L CNN
 F 1 "1u" H 7592 3355 50  0000 L CNN
 F 2 "Capacitor_SMD:C_1206_3216Metric" H 7500 3400 50  0001 C CNN
@@
 	7150 3450 7150 3650
 $Comp
-L Device:C_Small C24
+L Device:C_Small C26
 U 1 1 601E809B
 P 7300 3500
-F 0 "C24" H 7392 3546 50  0000 L CNN
+F 0 "C26" H 7392 3546 50  0000 L CNN
 F 1 "1u" H 7392 3455 50  0000 L CNN
 F 2 "Capacitor_SMD:C_1206_3216Metric" H 7300 3500 50  0001 C CNN
@@
 	7750 3650 7750 3500
 $Comp
-L Device:C_Small C26
+L Device:C_Small C28
 U 1 1 6023E9B3
 P 7750 3400
-F 0 "C26" H 7842 3446 50  0000 L CNN
+F 0 "C28" H 7842 3446 50  0000 L CNN
 F 1 "1u" H 7842 3355 50  0000 L CNN
 F 2 "Capacitor_SMD:C_1206_3216Metric" H 7750 3400 50  0001 C CNN
@@
 	7450 3050 7450 2900
 $Comp
-L Device:C_Small C27
+L Device:C_Small C29
 U 1 1 602D5887
 P 8100 2600
-F 0 "C27" V 8329 2600 50  0000 C CNN
+F 0 "C29" V 8329 2600 50  0000 C CNN
 F 1 "0.1u" V 8238 2600 50  0000 C CNN
-F 2 "Capacitor_SMD:C_1206_3216Metric" H 8100 2600 50  0001 C CNN
+F 2 "Capacitor_SMD:C_0603_1608Metric" H 8100 2600 50  0001 C CNN
 F 3 "~" H 8100 2600 50  0001 C CNN
 	1    8100 2600
@@
 F 3 "" H 8350 2600 50  0001 C CNN
 	1    8350 2600
-	0    -1   -1   0
+	1    0    0    -1
 $EndComp
 Wire Wire Line
@@
 Wire Wire Line
 	7100 1950 7100 2050
-Wire Wire Line
-	6450 1650 6450 1600
 Connection ~ 6450 1650
 Wire Wire Line
@@
 L power:GND #PWR044
 U 1 1 604A2D56
-P 6450 1600
-F 0 "#PWR044" H 6450 1350 50  0001 C CNN
-F 1 "GND" H 6455 1427 50  0000 C CNN
-F 2 "" H 6450 1600 50  0001 C CNN
-F 3 "" H 6450 1600 50  0001 C CNN
-	1    6450 1600
-	-1   0    0    1
+P 6550 1500
+F 0 "#PWR044" H 6550 1250 50  0001 C CNN
+F 1 "GND" H 6555 1327 50  0000 C CNN
+F 2 "" H 6550 1500 50  0001 C CNN
+F 3 "" H 6550 1500 50  0001 C CNN
+	1    6550 1500
+	1    0    0    -1
 $EndComp
 Wire Wire Line
@@
 	4750 1700 5650 1700
 $Comp
-L Device:C_Small C23
+L Device:C_Small C25
 U 1 1 6051CA4B
 P 4750 1850
-F 0 "C23" H 4842 1896 50  0000 L CNN
+F 0 "C25" H 4842 1896 50  0000 L CNN
 F 1 "1u" H 4842 1805 50  0000 L CNN
 F 2 "Capacitor_SMD:C_1206_3216Metric" H 4750 1850 50  0001 C CNN
@@
 	8200 2600 8350 2600
 $Comp
-L LTC6810-1:LTC6810-1-LTC6810-1 LTC1
+L LTC6810-1:LTC6810-1-LTC6810-1 LTC?
 U 1 1 5FF8D74A
 P 7350 4100
-AR Path="/5FF8D74A" Ref="LTC1"  Part="1"
+AR Path="/5FF8D74A" Ref="LTC?"  Part="1"
 AR Path="/5FF86554/5FF8D74A" Ref="LTC1"  Part="1"
 F 0 "LTC1" H 6450 6475 50  0000 C CNN
@@
 	0    -1   -1   0
 $EndComp
+Wire Wire Line
+	6550 1500 6450 1500
+Wire Wire Line
+	6450 1500 6450 1650
 $EndSCHEMATC

Commit message: ZCO version
Connections:
- net GND: no longer BT5.2 (-), BT6.1 (+), D14.2 (A), J11.1 (Pin_1), Q7.2 (S), R16.1, R22.2, R28.1
- new net: BT5.2 (-), BT6.1 (+), D14.2 (A), J11.1 (Pin_1), Q7.2 (S), R16.1, R22.2, R28.1
Changed lines of the file:
@@
 Wire Wire Line
 	5350 8550 5350 3450
-Wire Wire Line
-	3600 8550 3850 8550
-Wire Wire Line
-	3600 8550 3600 8600
-Connection ~ 3600 8550
 Connection ~ 3600 9600
 Wire Wire Line
@@
 	4100 9050 4100 8850
 Connection ~ 4100 9050
-Wire Wire Line
-	3200 8550 3600 8550
-Connection ~ 3200 8550
 Wire Wire Line
 	3050 8550 3200 8550
@@
 	4250 6450 5150 6450
 Wire Wire Line
-	5150 3050 5150 6450
-Wire Wire Line
 	4100 5900 5100 5900
 Wire Wire Line
-	5100 2950 5100 5900
-Wire Wire Line
 	4250 5400 5050 5400
 Wire Wire Line
-	5050 5400 5050 2850
-Wire Wire Line
-	4100 4850 5000 4850
-Wire Wire Line
 	5000 4850 5000 2750
 Wire Wire Line
-	4250 4350 4950 4350
-Wire Wire Line
 	4950 4350 4950 2650
-Wire Wire Line
-	4100 3800 4900 3800
 Wire Wire Line
 	4900 3800 4900 2550
@@
 	3050 8550 3050 8200
 Connection ~ 3600 8450
-Wire Wire Line
-	3600 8450 3600 8550
 Wire Wire Line
 	4100 8000 4100 8350
@@
 Connection ~ 3600 5300
 Wire Wire Line
-	4100 4850 4100 5200
-Wire Wire Line
-	4100 4850 4100 4650
-Connection ~ 4100 4850
-Wire Wire Line
 	3200 4350 3850 4350
 Connection ~ 3200 4350
@@
 Wire Wire Line
 	3600 5050 3600 5100
-$Comp
-L power:GND #PWR037
-U 1 1 600FD82C
-P 4250 4600
-F 0 "#PWR037" H 4250 4350 50  0001 C CNN
-F 1 "GND" H 4255 4427 50  0000 C CNN
-F 2 "" H 4250 4600 50  0001 C CNN
-F 3 "" H 4250 4600 50  0001 C CNN
-	1    4250 4600
-	1    0    0    -1
-$EndComp
 Wire Wire Line
 	4250 4550 4250 4600
 Wire Wire Line
 	3050 4350 3050 4750
-Connection ~ 4250 4350
 $Comp
 L Device:R_Small R25
@@
 	4050 4350 4250 4350
 $Comp
-L Device:C_Small C19
-U 1 1 600FD81B
-P 4250 4450
-F 0 "C19" H 4158 4404 50  0000 R CNN
-F 1 "10nF" H 4158 4495 50  0000 R CNN
-F 2 "Capacitor_SMD:C_1206_3216Metric" H 4250 4450 50  0001 C CNN
-F 3 "~" H 4250 4450 50  0001 C CNN
-	1    4250 4450
-	-1   0    0    1
-$EndComp
-$Comp
 L Device:Battery_Cell BT3
 U 1 1 600FD815
@@
 	3050 4350 3050 4000
 Connection ~ 3600 4250
-Wire Wire Line
-	4100 3800 4100 4150
-Wire Wire Line
-	4100 3800 4100 3600
-Connection ~ 4100 3800
 Wire Wire Line
 	4100 2750 4100 3100
@@
 Wire Wire Line
 	3600 4000 3600 4050
-$Comp
-L power:GND #PWR036
-U 1 1 5FFC24FD
-P 4250 3550
-F 0 "#PWR036" H 4250 3300 50  0001 C CNN
-F 1 "GND" H 4255 3377 50  0000 C CNN
-F 2 "" H 4250 3550 50  0001 C CNN
-F 3 "" H 4250 3550 50  0001 C CNN
-	1    4250 3550
-	1    0    0    -1
-$EndComp
 Wire Wire Line
 	4250 3500 4250 3550
@@
 Wire Wire Line
 	6450 1500 6450 1650
+Connection ~ 4100 3800
+Wire Wire Line
+	4100 3800 4100 3600
+Wire Wire Line
+	4100 3800 4100 4150
+Connection ~ 4250 4350
+Connection ~ 4100 4850
+Wire Wire Line
+	4100 4850 4100 4650
+Wire Wire Line
+	4100 4850 4100 5200
+Wire Wire Line
+	5150 3050 5150 6450
+Wire Wire Line
+	5100 2950 5100 5900
+Wire Wire Line
+	5050 5400 5050 2850
+$Comp
+L power:GND #PWR036
+U 1 1 5FFC24FD
+P 4250 3550
+F 0 "#PWR036" H 4250 3300 50  0001 C CNN
+F 1 "GND" H 4255 3377 50  0000 C CNN
+F 2 "" H 4250 3550 50  0001 C CNN
+F 3 "" H 4250 3550 50  0001 C CNN
+	1    4250 3550
+	1    0    0    -1
+$EndComp
+$Comp
+L Device:C_Small C19
+U 1 1 600FD81B
+P 4250 4450
+F 0 "C19" H 4158 4404 50  0000 R CNN
+F 1 "10nF" H 4158 4495 50  0000 R CNN
+F 2 "Capacitor_SMD:C_1206_3216Metric" H 4250 4450 50  0001 C CNN
+F 3 "~" H 4250 4450 50  0001 C CNN
+	1    4250 4450
+	-1   0    0    1
+$EndComp
+$Comp
+L power:GND #PWR037
+U 1 1 600FD82C
+P 4250 4600
+F 0 "#PWR037" H 4250 4350 50  0001 C CNN
+F 1 "GND" H 4255 4427 50  0000 C CNN
+F 2 "" H 4250 4600 50  0001 C CNN
+F 3 "" H 4250 4600 50  0001 C CNN
+	1    4250 4600
+	1    0    0    -1
+$EndComp
+Wire Wire Line
+	4100 3800 4900 3800
+Wire Wire Line
+	4250 4350 4950 4350
+Wire Wire Line
+	4100 4850 5000 4850
+Wire Wire Line
+	3600 8450 3600 8600
+Wire Wire Line
+	3200 8550 3850 8550
+Connection ~ 3200 8550
 $EndSCHEMATC

Commit message: Going back to work
Connections:
- net GND: now also BT5.2 (-), BT6.1 (+), D14.2 (A), J11.1 (Pin_1), Q7.2 (S), R16.1, R22.2, R28.1
Changed lines of the file:
@@
 Wire Wire Line
 	5350 8550 5350 3450
+Wire Wire Line
+	3600 8550 3850 8550
+Wire Wire Line
+	3600 8550 3600 8600
+Connection ~ 3600 8550
 Connection ~ 3600 9600
 Wire Wire Line
@@
 	4100 9050 4100 8850
 Connection ~ 4100 9050
+Wire Wire Line
+	3200 8550 3600 8550
+Connection ~ 3200 8550
 Wire Wire Line
 	3050 8550 3200 8550
@@
 	4250 6450 5150 6450
 Wire Wire Line
+	5150 3050 5150 6450
+Wire Wire Line
 	4100 5900 5100 5900
 Wire Wire Line
+	5100 2950 5100 5900
+Wire Wire Line
 	4250 5400 5050 5400
 Wire Wire Line
+	5050 5400 5050 2850
+Wire Wire Line
+	4100 4850 5000 4850
+Wire Wire Line
 	5000 4850 5000 2750
 Wire Wire Line
+	4250 4350 4950 4350
+Wire Wire Line
 	4950 4350 4950 2650
+Wire Wire Line
+	4100 3800 4900 3800
 Wire Wire Line
 	4900 3800 4900 2550
@@
 	3050 8550 3050 8200
 Connection ~ 3600 8450
+Wire Wire Line
+	3600 8450 3600 8550
 Wire Wire Line
 	4100 8000 4100 8350
@@
 Connection ~ 3600 5300
 Wire Wire Line
+	4100 4850 4100 5200
+Wire Wire Line
+	4100 4850 4100 4650
+Connection ~ 4100 4850
+Wire Wire Line
 	3200 4350 3850 4350
 Connection ~ 3200 4350
@@
 Wire Wire Line
 	3600 5050 3600 5100
+$Comp
+L power:GND #PWR037
+U 1 1 600FD82C
+P 4250 4600
+F 0 "#PWR037" H 4250 4350 50  0001 C CNN
+F 1 "GND" H 4255 4427 50  0000 C CNN
+F 2 "" H 4250 4600 50  0001 C CNN
+F 3 "" H 4250 4600 50  0001 C CNN
+	1    4250 4600
+	1    0    0    -1
+$EndComp
 Wire Wire Line
 	4250 4550 4250 4600
 Wire Wire Line
 	3050 4350 3050 4750
+Connection ~ 4250 4350
 $Comp
 L Device:R_Small R25
@@
 	4050 4350 4250 4350
 $Comp
+L Device:C_Small C19
+U 1 1 600FD81B
+P 4250 4450
+F 0 "C19" H 4158 4404 50  0000 R CNN
+F 1 "10nF" H 4158 4495 50  0000 R CNN
+F 2 "Capacitor_SMD:C_1206_3216Metric" H 4250 4450 50  0001 C CNN
+F 3 "~" H 4250 4450 50  0001 C CNN
+	1    4250 4450
+	-1   0    0    1
+$EndComp
+$Comp
 L Device:Battery_Cell BT3
 U 1 1 600FD815
@@
 	3050 4350 3050 4000
 Connection ~ 3600 4250
+Wire Wire Line
+	4100 3800 4100 4150
+Wire Wire Line
+	4100 3800 4100 3600
+Connection ~ 4100 3800
 Wire Wire Line
 	4100 2750 4100 3100
@@
 Wire Wire Line
 	3600 4000 3600 4050
+$Comp
+L power:GND #PWR036
+U 1 1 5FFC24FD
+P 4250 3550
+F 0 "#PWR036" H 4250 3300 50  0001 C CNN
+F 1 "GND" H 4255 3377 50  0000 C CNN
+F 2 "" H 4250 3550 50  0001 C CNN
+F 3 "" H 4250 3550 50  0001 C CNN
+	1    4250 3550
+	1    0    0    -1
+$EndComp
 Wire Wire Line
 	4250 3500 4250 3550
@@
 Wire Wire Line
 	6450 1500 6450 1650
-Connection ~ 4100 3800
-Wire Wire Line
-	4100 3800 4100 3600
-Wire Wire Line
-	4100 3800 4100 4150
-Connection ~ 4250 4350
-Connection ~ 4100 4850
-Wire Wire Line
-	4100 4850 4100 4650
-Wire Wire Line
-	4100 4850 4100 5200
-Wire Wire Line
-	5150 3050 5150 6450
-Wire Wire Line
-	5100 2950 5100 5900
-Wire Wire Line
-	5050 5400 5050 2850
-$Comp
-L power:GND #PWR036
-U 1 1 5FFC24FD
-P 4250 3550
-F 0 "#PWR036" H 4250 3300 50  0001 C CNN
-F 1 "GND" H 4255 3377 50  0000 C CNN
-F 2 "" H 4250 3550 50  0001 C CNN
-F 3 "" H 4250 3550 50  0001 C CNN
-	1    4250 3550
-	1    0    0    -1
-$EndComp
-$Comp
-L Device:C_Small C19
-U 1 1 600FD81B
-P 4250 4450
-F 0 "C19" H 4158 4404 50  0000 R CNN
-F 1 "10nF" H 4158 4495 50  0000 R CNN
-F 2 "Capacitor_SMD:C_1206_3216Metric" H 4250 4450 50  0001 C CNN
-F 3 "~" H 4250 4450 50  0001 C CNN
-	1    4250 4450
-	-1   0    0    1
-$EndComp
-$Comp
-L power:GND #PWR037
-U 1 1 600FD82C
-P 4250 4600
-F 0 "#PWR037" H 4250 4350 50  0001 C CNN
-F 1 "GND" H 4255 4427 50  0000 C CNN
-F 2 "" H 4250 4600 50  0001 C CNN
-F 3 "" H 4250 4600 50  0001 C CNN
-	1    4250 4600
-	1    0    0    -1
-$EndComp
-Wire Wire Line
-	4100 3800 4900 3800
-Wire Wire Line
-	4250 4350 4950 4350
-Wire Wire Line
-	4100 4850 5000 4850
-Wire Wire Line
-	3600 8450 3600 8600
-Wire Wire Line
-	3200 8550 3850 8550
-Connection ~ 3200 8550
 $EndSCHEMATC

Commit message: pcb layout nearly done
Parts:
- added D17, D18, D19, D20, D21, D22, D23: LED_Small, LED_SMD:LED_0805_2012Metric, symbol Device:LED_Small
- added R41, R42, R43, R44, R45, R46, R47: 330, Resistor_SMD:R_1206_3216Metric, symbol Device:R_Small
- J10, J11, J12, J6, J7, J8, J9: footprint Connector_Pin:Pin_D1.0mm_L10.0mm_LooseFit -> CellPad:CellPad
- R10, R11, R12, R13, R14, R15, R16: footprint Resistor_SMD:R_1206_3216Metric -> Resistor_SMD:R_2512_6332Metric
Connections:
- net GND: no longer BT5.2 (-), BT6.1 (+), D14.2 (A), J11.1 (Pin_1), Q7.2 (S), R16.1, R22.2, R28.1
- net at BT1.1 (+), D9.2 (A), J6.1 (Pin_1)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: now also R41.2, R42.2
- net at Q2.3 (D), R10.2: now also D17.1 (K)
- net at BT1.2 (-), BT2.1 (+), D10.2 (A)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: now also R43.2
- net at Q3.3 (D), R11.2: now also D18.1 (K)
- net at BT2.2 (-), BT3.1 (+), D11.2 (A)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: now also R44.2
- net at BT3.2 (-), BT4.1 (+), D12.2 (A)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: now also R45.2
- net at Q4.3 (D), R12.2: now also D19.1 (K)
- net at BT4.2 (-), BT5.1 (+), D13.2 (A)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: now also R46.2
- net at Q5.3 (D), R13.2: now also D20.1 (K)
- net at Q6.3 (D), R14.2: now also D21.1 (K)
- net at Q7.3 (D), R15.2: now also D22.1 (K)
- net at Q8.3 (D), R16.2: now also D23.1 (K)
- new net: BT5.2 (-), BT6.1 (+), D14.2 (A), J11.1 (Pin_1), Q7.2 (S), R16.1, R22.2, R28.1, R47.2
- new net: D18.2 (A), R42.1
- new net: D17.2 (A), R41.1
- new net: D19.2 (A), R43.1
- new net: D20.2 (A), R44.1
- new net: D21.2 (A), R45.1
- new net: D22.2 (A), R46.1
- new net: D23.2 (A), R47.1
Other:
- moved on the sheet: R24, R25, R26, R27, R28, R29

Commit message: PCB layout v1
Parts:
- added R48, R49, R50, R51: 10k, Resistor_SMD:R_0805_2012Metric, symbol Device:R_Small
Connections:
- net GND: now also R48.1, R49.1, R50.1, R51.1; no longer LTC1.34 (IBIAS), LTC1.35 (ICMP), LTC1.38 (IMB), LTC1.39 (IPB)
- new net: LTC1.34 (IBIAS), R51.2
- new net: LTC1.35 (ICMP), R50.2
- new net: LTC1.38 (IMB), R49.2
- new net: LTC1.39 (IPB), R48.2
Other:
- moved on the sheet: C29, Q9, R32
Changed lines of the file:
@@
 EESchema Schematic File Version 4
-LIBS:bmsLV-cache
 EELAYER 30 0
 EELAYER END
@@
 Wire Wire Line
 	7750 3150 7750 3300
-Connection ~ 7750 3150
 Connection ~ 7750 3650
-Wire Wire Line
-	7050 3050 7450 3050
 $Comp
 L Device:Q_NPN_BCE Q9
 U 1 1 602887F0
-P 7650 2900
-F 0 "Q9" H 7841 2946 50  0000 L CNN
-F 1 "Q_NPN_BCE" H 7841 2855 50  0000 L CNN
-F 2 "Package_TO_SOT_SMD:SOT-23W" H 7850 3000 50  0001 C CNN
-F 3 "~" H 7650 2900 50  0001 C CNN
-	1    7650 2900
-	1    0    0    -1
-$EndComp
-Wire Wire Line
-	7750 3100 7750 3150
-Wire Wire Line
-	7450 3050 7450 2900
+P 8200 2900
+F 0 "Q9" H 8391 2946 50  0000 L CNN
+F 1 "Q_NPN_BCE" H 8391 2855 50  0000 L CNN
+F 2 "Package_TO_SOT_SMD:SOT-23W" H 8400 3000 50  0001 C CNN
+F 3 "~" H 8200 2900 50  0001 C CNN
+	1    8200 2900
+	1    0    0    -1
+$EndComp
+Wire Wire Line
+	8000 3050 8000 2900
 $Comp
 L Device:C_Small C29
 U 1 1 602D5887
-P 8100 2600
-F 0 "C29" V 8329 2600 50  0000 C CNN
-F 1 "0.1u" V 8238 2600 50  0000 C CNN
-F 2 "Capacitor_SMD:C_0603_1608Metric" H 8100 2600 50  0001 C CNN
-F 3 "~" H 8100 2600 50  0001 C CNN
-	1    8100 2600
+P 8650 2600
+F 0 "C29" V 8879 2600 50  0000 C CNN
+F 1 "0.1u" V 8788 2600 50  0000 C CNN
+F 2 "Capacitor_SMD:C_0603_1608Metric" H 8650 2600 50  0001 C CNN
+F 3 "~" H 8650 2600 50  0001 C CNN
+	1    8650 2600
 	0    -1   -1   0
 $EndComp
-Connection ~ 7750 2600
-Wire Wire Line
-	7750 2600 7750 2700
+Connection ~ 8300 2600
+Wire Wire Line
+	8300 2600 8300 2700
 $Comp
 L power:GND #PWR051
 U 1 1 60321616
-P 8350 2600
-F 0 "#PWR051" H 8350 2350 50  0001 C CNN
-F 1 "GND" V 8355 2472 50  0000 R CNN
-F 2 "" H 8350 2600 50  0001 C CNN
-F 3 "" H 8350 2600 50  0001 C CNN
-	1    8350 2600
-	1    0    0    -1
-$EndComp
-Wire Wire Line
-	7750 2300 7750 2600
+P 8900 2600
+F 0 "#PWR051" H 8900 2350 50  0001 C CNN
+F 1 "GND" V 8905 2472 50  0000 R CNN
+F 2 "" H 8900 2600 50  0001 C CNN
+F 3 "" H 8900 2600 50  0001 C CNN
+	1    8900 2600
+	1    0    0    -1
+$EndComp
+Wire Wire Line
+	8300 2300 8300 2600
 $Comp
 L Device:R_Small R32
 U 1 1 60331F67
-P 7750 2200
-F 0 "R32" H 7809 2246 50  0000 L CNN
-F 1 "100" H 7809 2155 50  0000 L CNN
-F 2 "Resistor_SMD:R_1206_3216Metric" H 7750 2200 50  0001 C CNN
-F 3 "~" H 7750 2200 50  0001 C CNN
-	1    7750 2200
+P 8300 2200
+F 0 "R32" H 8359 2246 50  0000 L CNN
+F 1 "100" H 8359 2155 50  0000 L CNN
+F 2 "Resistor_SMD:R_1206_3216Metric" H 8300 2200 50  0001 C CNN
+F 3 "~" H 8300 2200 50  0001 C CNN
+	1    8300 2200
 	1    0    0    -1
 $EndComp
@@
 Wire Wire Line
 	3850 2250 3850 1700
-Wire Wire Line
-	3850 1350 7750 1350
 Connection ~ 3850 2250
 Wire Wire Line
 	3850 2250 4050 2250
 Wire Wire Line
-	7750 1350 7750 2100
+	8300 1350 8300 2100
 Wire Wire Line
 	3850 1700 4250 1700
@@
 L power:GND #PWR046
 U 1 1 605E56B3
-P 7050 2450
-F 0 "#PWR046" H 7050 2200 50  0001 C CNN
-F 1 "GND" V 7055 2322 50  0000 R CNN
-F 2 "" H 7050 2450 50  0001 C CNN
-F 3 "" H 7050 2450 50  0001 C CNN
-	1    7050 2450
-	0    -1   -1   0
-$EndComp
-Wire Wire Line
-	7750 2600 8000 2600
-Wire Wire Line
-	8200 2600 8350 2600
+P 7600 2450
+F 0 "#PWR046" H 7600 2200 50  0001 C CNN
+F 1 "GND" V 7605 2322 50  0000 R CNN
+F 2 "" H 7600 2450 50  0001 C CNN
+F 3 "" H 7600 2450 50  0001 C CNN
+	1    7600 2450
+	1    0    0    -1
+$EndComp
+Wire Wire Line
+	8300 2600 8550 2600
+Wire Wire Line
+	8750 2600 8900 2600
 $Comp
 L LTC6810-1:LTC6810-1-LTC6810-1 LTC?
@@
 L power:GND #PWR047
 U 1 1 605F8879
-P 7050 2550
-F 0 "#PWR047" H 7050 2300 50  0001 C CNN
-F 1 "GND" V 7055 2422 50  0000 R CNN
-F 2 "" H 7050 2550 50  0001 C CNN
-F 3 "" H 7050 2550 50  0001 C CNN
-	1    7050 2550
-	0    -1   -1   0
+P 7550 2550
+F 0 "#PWR047" H 7550 2300 50  0001 C CNN
+F 1 "GND" V 7555 2422 50  0000 R CNN
+F 2 "" H 7550 2550 50  0001 C CNN
+F 3 "" H 7550 2550 50  0001 C CNN
+	1    7550 2550
+	1    0    0    -1
 $EndComp
 $Comp
 L power:GND #PWR048
 U 1 1 605F8ED2
-P 7050 2850
-F 0 "#PWR048" H 7050 2600 50  0001 C CNN
-F 1 "GND" V 7055 2722 50  0000 R CNN
-F 2 "" H 7050 2850 50  0001 C CNN
-F 3 "" H 7050 2850 50  0001 C CNN
-	1    7050 2850
-	0    -1   -1   0
+P 7600 2850
+F 0 "#PWR048" H 7600 2600 50  0001 C CNN
+F 1 "GND" V 7605 2722 50  0000 R CNN
+F 2 "" H 7600 2850 50  0001 C CNN
+F 3 "" H 7600 2850 50  0001 C CNN
+	1    7600 2850
+	1    0    0    -1
 $EndComp
 $Comp
 L power:GND #PWR049
 U 1 1 605F9ECA
-P 7050 2950
-F 0 "#PWR049" H 7050 2700 50  0001 C CNN
-F 1 "GND" V 7055 2822 50  0000 R CNN
-F 2 "" H 7050 2950 50  0001 C CNN
-F 3 "" H 7050 2950 50  0001 C CNN
-	1    7050 2950
-	0    -1   -1   0
+P 7550 2950
+F 0 "#PWR049" H 7550 2700 50  0001 C CNN
+F 1 "GND" V 7555 2822 50  0000 R CNN
+F 2 "" H 7550 2950 50  0001 C CNN
+F 3 "" H 7550 2950 50  0001 C CNN
+	1    7550 2950
+	1    0    0    -1
 $EndComp
 Wire Wire Line
@@
 	0    1    1    0
 $EndComp
+$Comp
+L Device:R_Small R48
+U 1 1 60413195
+P 7300 2450
+F 0 "R48" V 7104 2450 50  0000 C CNN
+F 1 "10k" V 7195 2450 50  0000 C CNN
+F 2 "Resistor_SMD:R_0805_2012Metric" H 7300 2450 50  0001 C CNN
+F 3 "~" H 7300 2450 50  0001 C CNN
+	1    7300 2450
+	0    1    1    0
+$EndComp
+$Comp
+L Device:R_Small R49
+U 1 1 60413B7A
+P 7300 2550
+F 0 "R49" V 7104 2550 50  0000 C CNN
+F 1 "10k" V 7195 2550 50  0000 C CNN
+F 2 "Resistor_SMD:R_0805_2012Metric" H 7300 2550 50  0001 C CNN
+F 3 "~" H 7300 2550 50  0001 C CNN
+	1    7300 2550
+	0    1    1    0
+$EndComp
+Wire Wire Line
+	7050 2450 7200 2450
+Wire Wire Line
+	7050 2550 7200 2550
+Wire Wire Line
+	7400 2550 7550 2550
+Wire Wire Line
+	7400 2450 7600 2450
+Wire Wire Line
+	7050 3050 8000 3050
+Wire Wire Line
+	7750 3150 8300 3150
+Wire Wire Line
+	8300 3150 8300 3100
+Connection ~ 7750 3150
+$Comp
+L Device:R_Small R50
+U 1 1 6052A5A7
+P 7300 2850
+F 0 "R50" V 7104 2850 50  0000 C CNN
+F 1 "10k" V 7195 2850 50  0000 C CNN
+F 2 "Resistor_SMD:R_0805_2012Metric" H 7300 2850 50  0001 C CNN
+F 3 "~" H 7300 2850 50  0001 C CNN
+	1    7300 2850
+	0    1    1    0
+$EndComp
+$Comp
+L Device:R_Small R51
+U 1 1 6052CC05
+P 7300 2950
+F 0 "R51" V 7104 2950 50  0000 C CNN
+F 1 "10k" V 7195 2950 50  0000 C CNN
+F 2 "Resistor_SMD:R_0805_2012Metric" H 7300 2950 50  0001 C CNN
+F 3 "~" H 7300 2950 50  0001 C CNN
+	1    7300 2950
+	0    1    1    0
+$EndComp
+Wire Wire Line
+	7050 2850 7200 2850
+Wire Wire Line
+	7050 2950 7200 2950
+Wire Wire Line
+	7400 2950 7550 2950
+Wire Wire Line
+	7400 2850 7600 2850
+Wire Wire Line
+	3850 1350 8300 1350
 $EndSCHEMATC
