File: Hardware/bmsLV.sch (KiCad schematic (older format))
At the start: 28 parts, among them J1 Conn_01x06_Male, J2 USB_B_Mini, K1 RM85V7, Q1 BSS138, SW1 SW_Push, U1 STM32F103C8Tx, Y1 Crystal

Commit message: Power update
Parts:
- added J? (x2): Conn_01x02_Female, TerminalBlock:TerminalBlock_bornier-2_P5.08mm, symbol Connector:Conn_01x02_Female
Connections:
- net GND: now also J?.1 (Pin_1)
- new net CANH: J?.1 (Pin_1)
- new net CANL: J?.2 (Pin_2)
- new net VCC: J?.2 (Pin_2)
Other:
- moved on the sheet: J1, J2, K1, Q1, R7, R8

Commit message: Save before ZCO version
Parts:
- added D16: D_Small, Diode_SMD:D_SMB, symbol Device:D_Small
- added J13: Conn_01x04_Male, Connector_PinHeader_2.54mm:PinHeader_1x04_P2.54mm_Vertical, symbol Connector:Conn_01x04_Male
- K1: footprint RM85V7:RM85V7-Z-24VDC -> RM85V7:RM85V7
- gave numbers to parts that had none: 2
Connections:
- net +24V: now also D16.1 (K)
- net +5V: now also J13.1 (Pin_1)
- net GND: now also J13.4 (Pin_4)
- net USB_DM: now also J13.2 (Pin_2)
- net USB_DP: now also J13.3 (Pin_3)
- net at K1.2 (A2), Q1.3 (D): now also D16.2 (A)
Other:
- moved on the sheet: J2
Changed lines of the file:
@@
 L Connector:USB_B_Mini J2
 U 1 1 5FFA0FD0
-P 8150 1550
-F 0 "J2" H 7920 1447 50  0000 R CNN
-F 1 "USB_B_Mini" H 7920 1538 50  0000 R CNN
-F 2 "Connector_USB:USB_Micro-B_Molex_47346-0001" H 8300 1500 50  0001 C CNN
-F 3 "~" H 8300 1500 50  0001 C CNN
-	1    8150 1550
+P 8450 1550
+F 0 "J2" H 8220 1447 50  0000 R CNN
+F 1 "USB_B_Mini" H 8220 1538 50  0000 R CNN
+F 2 "Connector_USB:USB_Micro-B_Molex_47346-0001" H 8600 1500 50  0001 C CNN
+F 3 "~" H 8600 1500 50  0001 C CNN
+	1    8450 1550
 	-1   0    0    1
 $EndComp
@@
 L power:GND #PWR019
 U 1 1 5FFA2879
-P 8450 1100
-F 0 "#PWR019" H 8450 850 50  0001 C CNN
-F 1 "GND" H 8455 927 50  0000 C CNN
-F 2 "" H 8450 1100 50  0001 C CNN
-F 3 "" H 8450 1100 50  0001 C CNN
-	1    8450 1100
-	1    0    0    -1
-$EndComp
-Wire Wire Line
-	8150 1100 8150 1150
+P 8750 1100
+F 0 "#PWR019" H 8750 850 50  0001 C CNN
+F 1 "GND" H 8755 927 50  0000 C CNN
+F 2 "" H 8750 1100 50  0001 C CNN
+F 3 "" H 8750 1100 50  0001 C CNN
+	1    8750 1100
+	1    0    0    -1
+$EndComp
+Wire Wire Line
+	8450 1100 8450 1150
 $Comp
 L power:+5V #PWR014
 U 1 1 5FFAAF0D
-P 7450 1750
-F 0 "#PWR014" H 7450 1600 50  0001 C CNN
-F 1 "+5V" H 7465 1923 50  0000 C CNN
-F 2 "" H 7450 1750 50  0001 C CNN
-F 3 "" H 7450 1750 50  0001 C CNN
-	1    7450 1750
-	1    0    0    -1
-$EndComp
-Wire Wire Line
-	8150 1100 8250 1100
-Wire Wire Line
-	8250 1150 8250 1100
-Connection ~ 8250 1100
-Wire Wire Line
-	8250 1100 8450 1100
-Text GLabel 7850 1450 0    50   Input ~ 0
+P 7750 1750
+F 0 "#PWR014" H 7750 1600 50  0001 C CNN
+F 1 "+5V" H 7765 1923 50  0000 C CNN
+F 2 "" H 7750 1750 50  0001 C CNN
+F 3 "" H 7750 1750 50  0001 C CNN
+	1    7750 1750
+	1    0    0    -1
+$EndComp
+Wire Wire Line
+	8450 1100 8550 1100
+Wire Wire Line
+	8550 1150 8550 1100
+Connection ~ 8550 1100
+Wire Wire Line
+	8550 1100 8750 1100
+Text GLabel 8150 1450 0    50   Input ~ 0
 USB_DM
-Text GLabel 7850 1550 0    50   Input ~ 0
+Text GLabel 8150 1550 0    50   Input ~ 0
 USB_DP
 Wire Wire Line
-	7450 1750 7850 1750
+	7750 1750 8150 1750
 $Comp
 L power:+3.3V #PWR03
@@
 P 7900 2450
 AR Path="/5FAD7AC5/5FFFFAC2" Ref="J?"  Part="1"
-AR Path="/5FFFFAC2" Ref="J?"  Part="1"
-F 0 "J?" H 7792 2125 50  0000 C CNN
+AR Path="/5FFFFAC2" Ref="J3"  Part="1"
+F 0 "J3" H 7792 2125 50  0000 C CNN
 F 1 "Conn_01x02_Female" H 7792 2216 50  0000 C CNN
 F 2 "TerminalBlock:TerminalBlock_bornier-2_P5.08mm" H 7900 2450 50  0001 C CNN
@@
 P 8250 2450
 AR Path="/5FAD7AC5/5FFFFAC8" Ref="#PWR?"  Part="1"
-AR Path="/5FFFFAC8" Ref="#PWR?"  Part="1"
-F 0 "#PWR?" H 8250 2200 50  0001 C CNN
+AR Path="/5FFFFAC8" Ref="#PWR0101"  Part="1"
+F 0 "#PWR0101" H 8250 2200 50  0001 C CNN
 F 1 "GND" H 8255 2277 50  0000 C CNN
 F 2 "" H 8250 2450 50  0001 C CNN
@@
 	8250 2350 8250 2300
 $Comp
-L power:VCC #PWR?
+L power:VCC #PWR0102
 U 1 1 60004D86
 P 8250 2300
-F 0 "#PWR?" H 8250 2150 50  0001 C CNN
+F 0 "#PWR0102" H 8250 2150 50  0001 C CNN
 F 1 "VCC" H 8267 2473 50  0000 C CNN
 F 2 "" H 8250 2300 50  0001 C CNN
@@
 P 7900 3000
 AR Path="/5FB83FF2/60009E9A" Ref="J?"  Part="1"
-AR Path="/60009E9A" Ref="J?"  Part="1"
-F 0 "J?" H 7928 2976 50  0000 L CNN
+AR Path="/60009E9A" Ref="J5"  Part="1"
+F 0 "J5" H 7928 2976 50  0000 L CNN
 F 1 "Conn_01x02_Female" H 7928 2885 50  0000 L CNN
 F 2 "TerminalBlock:TerminalBlock_bornier-2_P5.08mm" H 7900 3000 50  0001 C CNN
@@
 F 0 "K1" H 8375 5475 50  0000 C CNN
 F 1 "RM85V7" H 8375 5384 50  0000 C CNN
-F 2 "RM85V7:RM85V7-Z-24VDC" V 8500 5200 50  0001 C CNN
+F 2 "RM85V7:RM85V7" V 8500 5200 50  0001 C CNN
 F 3 "" V 8500 5200 50  0001 C CNN
 	1    8350 5200
@@
 Wire Wire Line
 	8000 5350 8000 5600
-$Comp
-L Transistor_FET:BSS138 Q1
-U 1 1 60613319
-P 7900 5800
-F 0 "Q1" H 8105 5754 50  0000 L CNN
-F 1 "BSS138" H 8105 5845 50  0000 L CNN
-F 2 "Package_TO_SOT_SMD:SOT-23" H 8100 5725 50  0001 L CIN
-F 3 "https://www.fairchildsemi.com/datasheets/BS/BSS138.pdf" H 7900 5800 50  0001 L CNN
-	1    7900 5800
-	1    0    0    -1
-$EndComp
 $Comp
 L power:GND #PWR018
@@
 	1    0    0    -1
 $EndComp
+Wire Wire Line
+	8000 5350 7900 5350
+Wire Wire Line
+	7900 5150 8000 5150
+Connection ~ 8000 5350
+Connection ~ 8000 5150
+$Comp
+L Device:D_Small D16
+U 1 1 60308393
+P 7900 5250
+F 0 "D16" H 7900 5455 50  0000 C CNN
+F 1 "D_Small" H 7900 5364 50  0000 C CNN
+F 2 "Diode_SMD:D_SMB" V 7900 5250 50  0001 C CNN
+F 3 "~" V 7900 5250 50  0001 C CNN
+	1    7900 5250
+	0    1    1    0
+$EndComp
+$Comp
+L Transistor_FET:BSS138 Q1
+U 1 1 60613319
+P 7900 5800
+F 0 "Q1" H 8105 5754 50  0000 L CNN
+F 1 "BSS138" H 8105 5845 50  0000 L CNN
+F 2 "Package_TO_SOT_SMD:SOT-23" H 8100 5725 50  0001 L CIN
+F 3 "https://www.fairchildsemi.com/datasheets/BS/BSS138.pdf" H 7900 5800 50  0001 L CNN
+	1    7900 5800
+	1    0    0    -1
+$EndComp
+$Comp
+L Connector:Conn_01x04_Male J13
+U 1 1 60342BDE
+P 7000 1450
+F 0 "J13" H 7108 1731 50  0000 C CNN
+F 1 "Conn_01x04_Male" H 7108 1640 50  0000 C CNN
+F 2 "Connector_PinHeader_2.54mm:PinHeader_1x04_P2.54mm_Vertical" H 7000 1450 50  0001 C CNN
+F 3 "~" H 7000 1450 50  0001 C CNN
+	1    7000 1450
+	1    0    0    -1
+$EndComp
+$Comp
+L power:+5V #PWR0104
+U 1 1 6034A78E
+P 7200 1350
+F 0 "#PWR0104" H 7200 1200 50  0001 C CNN
+F 1 "+5V" H 7215 1523 50  0000 C CNN
+F 2 "" H 7200 1350 50  0001 C CNN
+F 3 "" H 7200 1350 50  0001 C CNN
+	1    7200 1350
+	1    0    0    -1
+$EndComp
+Text GLabel 7200 1450 2    50   Input ~ 0
+USB_DM
+Text GLabel 7200 1550 2    50   Input ~ 0
+USB_DP
+$Comp
+L power:GND #PWR0105
+U 1 1 60352852
+P 7200 1650
+F 0 "#PWR0105" H 7200 1400 50  0001 C CNN
+F 1 "GND" H 7205 1477 50  0000 C CNN
+F 2 "" H 7200 1650 50  0001 C CNN
+F 3 "" H 7200 1650 50  0001 C CNN
+	1    7200 1650
+	1    0    0    -1
+$EndComp

Commit message: Save before ZCO version- back
Parts:
- removed D16: D_Small, Diode_SMD:D_SMB, symbol Device:D_Small
- removed J13: Conn_01x04_Male, Connector_PinHeader_2.54mm:PinHeader_1x04_P2.54mm_Vertical, symbol Connector:Conn_01x04_Male
- K1: footprint RM85V7:RM85V7 -> RM85V7:RM85V7-Z-24VDC
- renumbered J3 to J?, J5 to J?
Other:
- moved on the sheet: J2
Changed lines of the file:
@@
 L Connector:USB_B_Mini J2
 U 1 1 5FFA0FD0
-P 8450 1550
-F 0 "J2" H 8220 1447 50  0000 R CNN
-F 1 "USB_B_Mini" H 8220 1538 50  0000 R CNN
-F 2 "Connector_USB:USB_Micro-B_Molex_47346-0001" H 8600 1500 50  0001 C CNN
-F 3 "~" H 8600 1500 50  0001 C CNN
-	1    8450 1550
+P 8150 1550
+F 0 "J2" H 7920 1447 50  0000 R CNN
+F 1 "USB_B_Mini" H 7920 1538 50  0000 R CNN
+F 2 "Connector_USB:USB_Micro-B_Molex_47346-0001" H 8300 1500 50  0001 C CNN
+F 3 "~" H 8300 1500 50  0001 C CNN
+	1    8150 1550
 	-1   0    0    1
 $EndComp
@@
 L power:GND #PWR019
 U 1 1 5FFA2879
-P 8750 1100
-F 0 "#PWR019" H 8750 850 50  0001 C CNN
-F 1 "GND" H 8755 927 50  0000 C CNN
-F 2 "" H 8750 1100 50  0001 C CNN
-F 3 "" H 8750 1100 50  0001 C CNN
-	1    8750 1100
-	1    0    0    -1
-$EndComp
-Wire Wire Line
-	8450 1100 8450 1150
+P 8450 1100
+F 0 "#PWR019" H 8450 850 50  0001 C CNN
+F 1 "GND" H 8455 927 50  0000 C CNN
+F 2 "" H 8450 1100 50  0001 C CNN
+F 3 "" H 8450 1100 50  0001 C CNN
+	1    8450 1100
+	1    0    0    -1
+$EndComp
+Wire Wire Line
+	8150 1100 8150 1150
 $Comp
 L power:+5V #PWR014
 U 1 1 5FFAAF0D
-P 7750 1750
-F 0 "#PWR014" H 7750 1600 50  0001 C CNN
-F 1 "+5V" H 7765 1923 50  0000 C CNN
-F 2 "" H 7750 1750 50  0001 C CNN
-F 3 "" H 7750 1750 50  0001 C CNN
-	1    7750 1750
-	1    0    0    -1
-$EndComp
-Wire Wire Line
-	8450 1100 8550 1100
-Wire Wire Line
-	8550 1150 8550 1100
-Connection ~ 8550 1100
-Wire Wire Line
-	8550 1100 8750 1100
-Text GLabel 8150 1450 0    50   Input ~ 0
+P 7450 1750
+F 0 "#PWR014" H 7450 1600 50  0001 C CNN
+F 1 "+5V" H 7465 1923 50  0000 C CNN
+F 2 "" H 7450 1750 50  0001 C CNN
+F 3 "" H 7450 1750 50  0001 C CNN
+	1    7450 1750
+	1    0    0    -1
+$EndComp
+Wire Wire Line
+	8150 1100 8250 1100
+Wire Wire Line
+	8250 1150 8250 1100
+Connection ~ 8250 1100
+Wire Wire Line
+	8250 1100 8450 1100
+Text GLabel 7850 1450 0    50   Input ~ 0
 USB_DM
-Text GLabel 8150 1550 0    50   Input ~ 0
+Text GLabel 7850 1550 0    50   Input ~ 0
 USB_DP
 Wire Wire Line
-	7750 1750 8150 1750
+	7450 1750 7850 1750
 $Comp
 L power:+3.3V #PWR03
@@
 P 7900 2450
 AR Path="/5FAD7AC5/5FFFFAC2" Ref="J?"  Part="1"
-AR Path="/5FFFFAC2" Ref="J3"  Part="1"
-F 0 "J3" H 7792 2125 50  0000 C CNN
+AR Path="/5FFFFAC2" Ref="J?"  Part="1"
+F 0 "J?" H 7792 2125 50  0000 C CNN
 F 1 "Conn_01x02_Female" H 7792 2216 50  0000 C CNN
 F 2 "TerminalBlock:TerminalBlock_bornier-2_P5.08mm" H 7900 2450 50  0001 C CNN
@@
 P 8250 2450
 AR Path="/5FAD7AC5/5FFFFAC8" Ref="#PWR?"  Part="1"
-AR Path="/5FFFFAC8" Ref="#PWR0101"  Part="1"
-F 0 "#PWR0101" H 8250 2200 50  0001 C CNN
+AR Path="/5FFFFAC8" Ref="#PWR?"  Part="1"
+F 0 "#PWR?" H 8250 2200 50  0001 C CNN
 F 1 "GND" H 8255 2277 50  0000 C CNN
 F 2 "" H 8250 2450 50  0001 C CNN
@@
 	8250 2350 8250 2300
 $Comp
-L power:VCC #PWR0102
+L power:VCC #PWR?
 U 1 1 60004D86
 P 8250 2300
-F 0 "#PWR0102" H 8250 2150 50  0001 C CNN
+F 0 "#PWR?" H 8250 2150 50  0001 C CNN
 F 1 "VCC" H 8267 2473 50  0000 C CNN
 F 2 "" H 8250 2300 50  0001 C CNN
@@
 P 7900 3000
 AR Path="/5FB83FF2/60009E9A" Ref="J?"  Part="1"
-AR Path="/60009E9A" Ref="J5"  Part="1"
-F 0 "J5" H 7928 2976 50  0000 L CNN
+AR Path="/60009E9A" Ref="J?"  Part="1"
+F 0 "J?" H 7928 2976 50  0000 L CNN
 F 1 "Conn_01x02_Female" H 7928 2885 50  0000 L CNN
 F 2 "TerminalBlock:TerminalBlock_bornier-2_P5.08mm" H 7900 3000 50  0001 C CNN
@@
 F 0 "K1" H 8375 5475 50  0000 C CNN
 F 1 "RM85V7" H 8375 5384 50  0000 C CNN
-F 2 "RM85V7:RM85V7" V 8500 5200 50  0001 C CNN
+F 2 "RM85V7:RM85V7-Z-24VDC" V 8500 5200 50  0001 C CNN
 F 3 "" V 8500 5200 50  0001 C CNN
 	1    8350 5200
@@
 Wire Wire Line
 	8000 5350 8000 5600
+$Comp
+L Transistor_FET:BSS138 Q1
+U 1 1 60613319
+P 7900 5800
+F 0 "Q1" H 8105 5754 50  0000 L CNN
+F 1 "BSS138" H 8105 5845 50  0000 L CNN
+F 2 "Package_TO_SOT_SMD:SOT-23" H 8100 5725 50  0001 L CIN
+F 3 "https://www.fairchildsemi.com/datasheets/BS/BSS138.pdf" H 7900 5800 50  0001 L CNN
+	1    7900 5800
+	1    0    0    -1
+$EndComp
 $Comp
 L power:GND #PWR018
@@
 	1    0    0    -1
 $EndComp
-Wire Wire Line
-	8000 5350 7900 5350
-Wire Wire Line
-	7900 5150 8000 5150
-Connection ~ 8000 5350
-Connection ~ 8000 5150
-$Comp
-L Device:D_Small D16
-U 1 1 60308393
-P 7900 5250
-F 0 "D16" H 7900 5455 50  0000 C CNN
-F 1 "D_Small" H 7900 5364 50  0000 C CNN
-F 2 "Diode_SMD:D_SMB" V 7900 5250 50  0001 C CNN
-F 3 "~" V 7900 5250 50  0001 C CNN
-	1    7900 5250
-	0    1    1    0
-$EndComp
-$Comp
-L Transistor_FET:BSS138 Q1
-U 1 1 60613319
-P 7900 5800
-F 0 "Q1" H 8105 5754 50  0000 L CNN
-F 1 "BSS138" H 8105 5845 50  0000 L CNN
-F 2 "Package_TO_SOT_SMD:SOT-23" H 8100 5725 50  0001 L CIN
-F 3 "https://www.fairchildsemi.com/datasheets/BS/BSS138.pdf" H 7900 5800 50  0001 L CNN
-	1    7900 5800
-	1    0    0    -1
-$EndComp
-$Comp
-L Connector:Conn_01x04_Male J13
-U 1 1 60342BDE
-P 7000 1450
-F 0 "J13" H 7108 1731 50  0000 C CNN
-F 1 "Conn_01x04_Male" H 7108 1640 50  0000 C CNN
-F 2 "Connector_PinHeader_2.54mm:PinHeader_1x04_P2.54mm_Vertical" H 7000 1450 50  0001 C CNN
-F 3 "~" H 7000 1450 50  0001 C CNN
-	1    7000 1450
-	1    0    0    -1
-$EndComp
-$Comp
-L power:+5V #PWR0104
-U 1 1 6034A78E
-P 7200 1350
-F 0 "#PWR0104" H 7200 1200 50  0001 C CNN
-F 1 "+5V" H 7215 1523 50  0000 C CNN
-F 2 "" H 7200 1350 50  0001 C CNN
-F 3 "" H 7200 1350 50  0001 C CNN
-	1    7200 1350
-	1    0    0    -1
-$EndComp
-Text GLabel 7200 1450 2    50   Input ~ 0
-USB_DM
-Text GLabel 7200 1550 2    50   Input ~ 0
-USB_DP
-$Comp
-L power:GND #PWR0105
-U 1 1 60352852
-P 7200 1650
-F 0 "#PWR0105" H 7200 1400 50  0001 C CNN
-F 1 "GND" H 7205 1477 50  0000 C CNN
-F 2 "" H 7200 1650 50  0001 C CNN
-F 3 "" H 7200 1650 50  0001 C CNN
-	1    7200 1650
-	1    0    0    -1
-$EndComp
