File: Hardware/Can.sch (KiCad schematic (older format))
At the start: 7 parts, among them J4 Conn_01x02_Male, J5 Conn_01x02_Female, U4 MCP2562-H-SN

Commit message: Power update
Parts:
- removed J5: Conn_01x02_Female, TerminalBlock:TerminalBlock_bornier-2_P5.08mm, symbol Connector:Conn_01x02_Female
- renumbered C14 to C16, C15 to C17
Changed lines of the file:
@@
 $EndComp
 $Comp
-L Device:C_Small C15
+L Device:C_Small C17
 U 1 1 5FB886F3
 P 3550 1800
-F 0 "C15" V 3321 1800 50  0000 C CNN
+F 0 "C17" V 3321 1800 50  0000 C CNN
 F 1 "100n" V 3412 1800 50  0000 C CNN
 F 2 "Capacitor_SMD:C_1206_3216Metric" H 3550 1800 50  0001 C CNN
@@
 F 3 "" H 3350 1800 50  0001 C CNN
 	1    3350 1800
-	0    1    1    0
+	1    0    0    -1
 $EndComp
 Wire Wire Line
@@
 $EndComp
 $Comp
-L Device:C_Small C14
+L Device:C_Small C16
 U 1 1 5FB8B717
 P 2900 2700
-F 0 "C14" V 2671 2700 50  0000 C CNN
+F 0 "C16" V 2671 2700 50  0000 C CNN
 F 1 "100n" V 2762 2700 50  0000 C CNN
 F 2 "Capacitor_SMD:C_1206_3216Metric" H 2900 2700 50  0001 C CNN
@@
 CANL
 $Comp
-L Connector:Conn_01x02_Female J5
-U 1 1 5FB9989C
-P 6600 2500
-F 0 "J5" H 6628 2476 50  0000 L CNN
-F 1 "Conn_01x02_Female" H 6628 2385 50  0000 L CNN
-F 2 "TerminalBlock:TerminalBlock_bornier-2_P5.08mm" H 6600 2500 50  0001 C CNN
-F 3 "~" H 6600 2500 50  0001 C CNN
-	1    6600 2500
-	1    0    0    -1
-$EndComp
-Text GLabel 6400 2500 0    50   Input ~ 0
-CANH
-Text GLabel 6400 2600 0    50   Input ~ 0
-CANL
-$Comp

Commit message: Software update 3
Current sensor added to PCB (through wires)
Current sensor handling added
Cell balance working! (HUGE PART OF UPDATE)
CheckError function modified (a lot of more error added)
Serial print function added (not tested)
+ some cosmetic changes
Parts:
- C16, C17: symbol Device:C_Small -> bmsLV-rescue:C_Small-Device
- D8: symbol Device:D_TVS_x2_AAC -> bmsLV-rescue:D_TVS_x2_AAC-Device
- J4: symbol Connector:Conn_01x02_Male -> bmsLV-rescue:Conn_01x02_Male-Connector
- R9: symbol Device:R_Small -> bmsLV-rescue:R_Small-Device
- U4: symbol Interface_CAN_LIN:MCP2562-H-SN -> bmsLV-rescue:MCP2562-H-SN-Interface_CAN_LIN
Changed lines of the file:
@@
 $EndDescr
 $Comp
-L Interface_CAN_LIN:MCP2562-H-SN U4
+L bmsLV-rescue:MCP2562-H-SN-Interface_CAN_LIN U4
 U 1 1 5FB847F4
 P 3650 2500
@@
 	3650 2100 3650 1800
 $Comp
-L power:+5V #PWR032
+L bmsLV-rescue:+5V-power #PWR032
 U 1 1 5FB87973
 P 3650 1650
@@
 $EndComp
 $Comp
-L Device:C_Small C17
+L bmsLV-rescue:C_Small-Device C17
 U 1 1 5FB886F3
 P 3550 1800
@@
 	3650 1800 3650 1650
 $Comp
-L power:GND #PWR031
+L bmsLV-rescue:GND-power #PWR031
 U 1 1 5FB8975D
 P 3350 1800
@@
 	3150 2600 2900 2600
 $Comp
-L power:+3.3V #PWR028
+L bmsLV-rescue:+3.3V-power #PWR028
 U 1 1 5FB8A58B
 P 2300 2600
@@
 $EndComp
 $Comp
-L Device:C_Small C16
+L bmsLV-rescue:C_Small-Device C16
 U 1 1 5FB8B717
 P 2900 2700
@@
 Connection ~ 2900 2600
 $Comp
-L power:GND #PWR029
+L bmsLV-rescue:GND-power #PWR029
 U 1 1 5FB8CC3F
 P 2900 2900
@@
 	3150 2700 3150 3000
 $Comp
-L power:GND #PWR030
+L bmsLV-rescue:GND-power #PWR030
 U 1 1 5FB8DCB8
 P 3150 3000
@@
 	3650 2900 3650 3000
 $Comp
-L power:GND #PWR033
+L bmsLV-rescue:GND-power #PWR033
 U 1 1 5FB9013B
 P 3650 3000
@@
 $EndComp
 $Comp
-L Device:R_Small R9
+L bmsLV-rescue:R_Small-Device R9
 U 1 1 5FB91F93
 P 4400 2400
@@
 	4400 2250 4400 2300
 $Comp
-L Device:D_TVS_x2_AAC D8
+L bmsLV-rescue:D_TVS_x2_AAC-Device D8
 U 1 1 5FB95EFA
 P 4800 2500
@@
 $EndComp
 $Comp
-L power:GND #PWR034
+L bmsLV-rescue:GND-power #PWR034
 U 1 1 5FB9744E
 P 5050 2500
@@
 CANL
 $Comp
-L Connector:Conn_01x02_Male J4
+L bmsLV-rescue:Conn_01x02_Male-Connector J4
 U 1 1 606A8AD6
 P 4600 2700
